Commit message: Fix Fortress-only URDF, physics, deps, scripts, and launch cleanup
- Normalize fdir1 to unit vectors (0.707107 ±0.707107 0)
- Sphere-only collision + correct sphere inertia tensor
- mu2=0.1, kp=200000, kd=2000 for stable contact on 50g wheels
- Ground plane mu=mu2=100 (symmetric, no strafe traction bias)
- Remove use_ignition everywhere; Fortress-only hardware plugin
- Fix load_ros2_controllers.launch.py: OnProcessStart + 2s delay
- Fix script/launch references to rosmaster_gazebo_fortress.launch.py
- RViz fixed frame: base_footprint
- package.xml: Classic → Fortress deps
- Re-enable controller load test with correct Humble ControllerManager API
- Fix docking launch PythonExpression string concat, add tf2 build dep
- Delete stale Classic launch files and ros2_controllers.yaml duplicate

Co-Authored-By: Claude Sonnet 4.6 <noreply@anthropic.com>

File: yahboom_rosmaster_description/urdf/control/rosmaster_x3_ros2_control.urdf.xacro (robot description, xacro)
@@ -1,13 +1,8 @@
 <?xml version="1.0" ?>
 <robot xmlns:xacro="http://wiki.ros.org/xacro">
-    <xacro:macro name="yahboom_rosmaster_ros2_control" params="prefix use_gazebo use_ignition:='false'">
+    <xacro:macro name="yahboom_rosmaster_ros2_control" params="prefix use_gazebo">
         <ros2_control name="RobotSystem" type="system">
             <hardware>
-                <xacro:if value="${use_ignition}">
-                    <plugin>gz_ros2_control/GazeboSimSystem</plugin>
-                </xacro:if>
-                <xacro:unless value="${use_ignition}">
-                    <plugin>gazebo_ros2_control/GazeboSystem</plugin>
-                </xacro:unless>
+                <plugin>gz_ros2_control/GazeboSimSystem</plugin>
             </hardware>
             <joint name="${prefix}front_left_wheel_joint">

File: yahboom_rosmaster_description/urdf/mech/mecanum_wheel.urdf.xacro (robot description, xacro)
@@ -7,5 +7,5 @@
   <xacro:property name="wheel_xoff" value="0.08" />
   <xacro:property name="wheel_yoff" value="-0.01" />
-  <xacro:macro name="mecanum_wheel" params="prefix side x_reflect y_reflect fdir1:='1 0 0' use_ignition:='false'">
+  <xacro:macro name="mecanum_wheel" params="prefix side x_reflect y_reflect fdir1:='0.707107 0 0'">
     <link name="${prefix}${side}_wheel_link">
       <visual>
@@ -18,29 +18,20 @@
         </material>
       </visual>
-      <!-- Fortress: sphere gives a single contact point, required for gz:expressed_in to work -->
-      <xacro:if value="${use_ignition}">
-        <collision>
-          <origin xyz="0 0 0" rpy="0 0 0"/>
-          <geometry>
-            <sphere radius="${wheel_radius}"/>
-          </geometry>
-        </collision>
-      </xacro:if>
-      <!-- Classic: cylinder collision (unchanged) -->
-      <xacro:unless value="${use_ignition}">
-        <collision>
-          <origin xyz="0 0 0" rpy="${pi/2} 0 0"/>
-          <geometry>
-            <cylinder radius="${wheel_radius}" length="${wheel_width}"/>
-          </geometry>
-        </collision>
-      </xacro:unless>
+      <!-- Sphere gives a single contact point, required for gz:expressed_in to lock fdir1 to chassis frame -->
+      <collision>
+        <origin xyz="0 0 0" rpy="0 0 0"/>
+        <geometry>
+          <sphere radius="${wheel_radius}"/>
+        </geometry>
+      </collision>
+      <!-- Sphere inertia: I = (2/5) * m * r^2 on all axes -->
       <inertial>
         <origin xyz="0 0 0" rpy="0 0 0"/>
         <mass value="${wheel_mass}"/>
+        <xacro:property name="I_sphere" value="${(2.0/5.0) * wheel_mass * wheel_radius * wheel_radius}"/>
         <inertia
-          ixx="${(wheel_mass/12.0) * (3*wheel_radius*wheel_radius + wheel_width*wheel_width)}" ixy="0" ixz="0"
-          iyy="${(wheel_mass/2.0) * (wheel_radius*wheel_radius)}" iyz="0"
-          izz="${(wheel_mass/12.0) * (3*wheel_radius*wheel_radius + wheel_width*wheel_width)}"/>
+          ixx="${I_sphere}" ixy="0" ixz="0"
+          iyy="${I_sphere}" iyz="0"
+          izz="${I_sphere}"/>
       </inertial>
     </link>
@@ -57,17 +48,16 @@
           <ode>
               <mu>1.0</mu>
-              <mu2>0.0</mu2>
-              <xacro:if value="${use_ignition}">
-                <fdir1 gz:expressed_in="${prefix}base_link">${fdir1}</fdir1>
-              </xacro:if>
-              <xacro:unless value="${use_ignition}">
-                <fdir1>${fdir1}</fdir1>
-              </xacro:unless>
+              <!-- mu2 small but non-zero to avoid contact instability at zero lateral friction -->
+              <mu2>0.1</mu2>
+              <!-- Lock fdir1 to chassis frame so roller direction stays correct as wheel spins -->
+              <fdir1 gz:expressed_in="${prefix}base_link">${fdir1}</fdir1>
           </ode>
         </friction>
         <contact>
           <ode>
-            <kp>1000000.0</kp>
-            <kd>100.0</kd>
+            <!-- Softer contact (was 1e6) reduces oscillations for 50g wheels -->
+            <kp>200000.0</kp>
+            <!-- kd/kp ≈ 0.01 prevents bounce -->
+            <kd>2000.0</kd>
             <min_depth>0.001</min_depth>
           </ode>

File: yahboom_rosmaster_description/urdf/robots/rosmaster_x3.urdf.xacro (robot description, xacro)
@@ -5,5 +5,4 @@
   <xacro:arg name="prefix" default=""/>
   <xacro:arg name="use_gazebo" default="false"/>
-  <xacro:arg name="use_ignition" default="false"/>
   <xacro:include filename="$(find yahboom_rosmaster_description)/urdf/mech/rosmaster_x3_base.urdf.xacro"/>
   <xacro:include filename="$(find yahboom_rosmaster_description)/urdf/mech/mecanum_wheel.urdf.xacro"/>
@@ -12,4 +11,7 @@
   <xacro:include filename="$(find yahboom_rosmaster_description)/urdf/sensors/imu.urdf.xacro"/>
   <xacro:rosmaster_x3_base prefix="$(arg prefix)"/>
+  <!-- fdir1 defines the roller axis direction (locked to chassis frame via gz:expressed_in).
+       FL/BR diagonal: rollers at -45° to forward  →  (1, -1, 0) normalized
+       FR/BL diagonal: rollers at +45° to forward  →  (1,  1, 0) normalized -->
   <xacro:mecanum_wheel
     prefix="$(arg prefix)"
@@ -17,6 +19,5 @@
     x_reflect="1"
     y_reflect="1"
-    fdir1="1 -1 0"
-    use_ignition="$(arg use_ignition)"/>
+    fdir1="0.707107 -0.707107 0"/>
   <xacro:mecanum_wheel
     prefix="$(arg prefix)"
@@ -24,6 +25,5 @@
     x_reflect="1"
     y_reflect="-1"
-    fdir1="1 1 0"
-    use_ignition="$(arg use_ignition)"/>
+    fdir1="0.707107 0.707107 0"/>
   <xacro:mecanum_wheel
     prefix="$(arg prefix)"
@@ -31,6 +31,5 @@
     x_reflect="-1"
     y_reflect="1"
-    fdir1="1 1 0"
-    use_ignition="$(arg use_ignition)"/>
+    fdir1="0.707107 0.707107 0"/>
   <xacro:mecanum_wheel
     prefix="$(arg prefix)"
@@ -38,6 +37,5 @@
     x_reflect="-1"
     y_reflect="-1"
-    fdir1="1 -1 0"
-    use_ignition="$(arg use_ignition)"/>
+    fdir1="0.707107 -0.707107 0"/>
   <xacro:rgbd_camera
     prefix="$(arg prefix)"
@@ -62,20 +60,11 @@
     update_rate="15.0"
     topic_name="imu/data"/>
-  <!-- Gazebo ros2_control plugin — Fortress (gz_ros2_control) or Classic (gazebo_ros2_control) -->
+  <!-- Gazebo Fortress ros2_control plugin (gz_ros2_control) -->
   <xacro:if value="$(arg use_gazebo)">
-    <xacro:if value="$(arg use_ignition)">
-      <gazebo>
-        <plugin filename="gz_ros2_control-system" name="gz_ros2_control::GazeboSimROS2ControlPlugin">
-          <parameters>$(find yahboom_rosmaster_gazebo)/config/ros2_control.yaml</parameters>
-        </plugin>
-      </gazebo>
-    </xacro:if>
-    <xacro:unless value="$(arg use_ignition)">
-      <gazebo>
-        <plugin name="gazebo_ros2_control" filename="libgazebo_ros2_control.so">
-          <parameters>$(find yahboom_rosmaster_gazebo)/config/ros2_control.yaml</parameters>
-        </plugin>
-      </gazebo>
-    </xacro:unless>
+    <gazebo>
+      <plugin filename="gz_ros2_control-system" name="gz_ros2_control::GazeboSimROS2ControlPlugin">
+        <parameters>$(find yahboom_rosmaster_gazebo)/config/ros2_control.yaml</parameters>
+      </plugin>
+    </gazebo>
   </xacro:if>
   <!-- ros2_control joints/interfaces for the robot -->
@@ -83,5 +72,4 @@
   <xacro:yahboom_rosmaster_ros2_control
     prefix="$(arg prefix)"
-    use_gazebo="$(arg use_gazebo)"
-    use_ignition="$(arg use_ignition)"/>
+    use_gazebo="$(arg use_gazebo)"/>
 </robot>

File: yahboom_rosmaster_description/urdf/sensors/rgbd_camera.urdf.xacro (robot description, xacro)
@@ -44,5 +44,5 @@
     update_rate:=2
     always_on:=1
-    visualize:=true
+    visualize:=false
     enable_collision:=false">
     <link name="${prefix}${camera_name}_link">

Commit message: Investigate mecanum strafing: document DART physics limitations
Reverted VelocityControl/passive-roller experiments; restored physics-based
approach (sphere collision + fdir1 + ignition:expressed_in="base_footprint").

Test results:
- Forward: Δx=+1.49m / 5s at 0.3 m/s (99% efficiency) ✓
- Rotation: CCW for angular.z=+0.5 ✓
- Strafe: BROKEN — produces -y for +y command + ~50° yaw rotation ✗

Root cause investigation:
- Passive rollers: DART LCP ignores passive joint DOF → isotropic → no strafe
- Bullet physics: doesn't support mu2/fdir1 → isotropic → no strafe
- fdir1+sphere: forward/rotation correct; strafing fails with any fdir1 assignment
  due to unknown DART + gz_ros2_control constraint interaction
- Official Gazebo mecanum demo (MecanumDrive plugin) strafes correctly with same
  fdir1 values — difference is MecanumDrive vs gz_ros2_control kinematic solver

Updated CLAUDE.md with detailed investigation findings and options for next session.

Co-Authored-By: Claude Sonnet 4.6 <noreply@anthropic.com>

File: yahboom_rosmaster_description/urdf/control/rosmaster_x3_ros2_control.urdf.xacro (robot description, xacro)
@@ -7,35 +7,23 @@
             </hardware>
             <joint name="${prefix}front_left_wheel_joint">
-              <command_interface name="velocity">
-                  <param name="min">-50.0</param>
-                  <param name="max">50.0</param>
-              </command_interface>
+              <command_interface name="velocity"/>
               <state_interface name="position"/>
               <state_interface name="velocity"/>
-          </joint>
-          <joint name="${prefix}front_right_wheel_joint">
-              <command_interface name="velocity">
-                  <param name="min">-50.0</param>
-                  <param name="max">50.0</param>
-              </command_interface>
+            </joint>
+            <joint name="${prefix}front_right_wheel_joint">
+              <command_interface name="velocity"/>
               <state_interface name="position"/>
               <state_interface name="velocity"/>
-          </joint>
-          <joint name="${prefix}back_left_wheel_joint">
-              <command_interface name="velocity">
-                  <param name="min">-50.0</param>
-                  <param name="max">50.0</param>
-              </command_interface>
+            </joint>
+            <joint name="${prefix}back_left_wheel_joint">
+              <command_interface name="velocity"/>
               <state_interface name="position"/>
               <state_interface name="velocity"/>
-          </joint>
-          <joint name="${prefix}back_right_wheel_joint">
-              <command_interface name="velocity">
-                  <param name="min">-50.0</param>
-                  <param name="max">50.0</param>
-              </command_interface>
+            </joint>
+            <joint name="${prefix}back_right_wheel_joint">
+              <command_interface name="velocity"/>
               <state_interface name="position"/>
               <state_interface name="velocity"/>
-          </joint>
+            </joint>
       </ros2_control>
   </xacro:macro>

File: yahboom_rosmaster_description/urdf/mech/mecanum_wheel.urdf.xacro (robot description, xacro)
@@ -1,10 +1,26 @@
 <?xml version="1.0"?>
-<robot xmlns:xacro="http://www.ros.org/wiki/xacro" xmlns:gz="http://gazebosim.org/schema">
-  <xacro:property name="wheel_radius" value="0.0325" />
-  <xacro:property name="wheel_separation" value="0.169" />
-  <xacro:property name="wheel_width" value="0.03040" />
-  <xacro:property name="wheel_mass" value="0.05" />  <!-- Real 65mm mecanum wheel ~40-60 g. Old 0.15 kg was 3× too heavy. -->
-  <xacro:property name="wheel_xoff" value="0.08" />
-  <xacro:property name="wheel_yoff" value="-0.01" />
+<!--
+  Mecanum wheel with sphere collision + fdir1 anisotropic friction.
+  Each wheel is a sphere (single contact point) with:
+    mu=1.0  along fdir1 (roller grip direction — high friction)
+    mu2=0.0 perpendicular to fdir1 (roller free-rolling direction — zero friction)
+  fdir1 is expressed in the robot base_link frame via ignition:expressed_in so
+  the friction direction rotates with the chassis at any heading.
+  With Bullet physics (ignition-physics5-bullet-plugin), expressed_in is
+  re-evaluated every physics step → correct holonomic motion at any heading.
+  With DART, expressed_in is computed once at model load (one-shot bug) → correct
+  strafing at initial yaw=0 only.
+  fdir1 values per wheel (set by caller in rosmaster_x3.urdf.xacro):
+    FL, BR: "0.707107 -0.707107 0"
+    FR, BL: "0.707107  0.707107 0"
+-->
+<robot xmlns:xacro="http://www.ros.org/wiki/xacro"
+       xmlns:ignition="http://ignitionrobotics.org/schema">
+  <xacro:property name="wheel_radius"    value="0.0325"  />
+  <xacro:property name="wheel_separation" value="0.169"  />
+  <xacro:property name="wheel_width"     value="0.03040" />
+  <xacro:property name="wheel_mass"      value="0.05"    />
+  <xacro:property name="wheel_xoff"      value="0.08"    />
+  <xacro:property name="wheel_yoff"      value="-0.01"   />
   <xacro:macro name="mecanum_wheel" params="prefix side x_reflect y_reflect fdir1:='0.707107 0 0'">
     <link name="${prefix}${side}_wheel_link">
@@ -18,5 +34,7 @@
         </material>
       </visual>
-      <!-- Sphere gives a single contact point, required for gz:expressed_in to lock fdir1 to chassis frame -->
+      <!-- Sphere gives a single contact point. Required for ignition:expressed_in
+           to correctly lock fdir1 to the chassis frame (cylinder gives an extended
+           contact line which behaves unpredictably with directional friction). -->
       <collision>
         <origin xyz="0 0 0" rpy="0 0 0"/>
@@ -25,13 +43,11 @@
         </geometry>
       </collision>
-      <!-- Sphere inertia: I = (2/5) * m * r^2 on all axes -->
       <inertial>
         <origin xyz="0 0 0" rpy="0 0 0"/>
         <mass value="${wheel_mass}"/>
         <xacro:property name="I_sphere" value="${(2.0/5.0) * wheel_mass * wheel_radius * wheel_radius}"/>
-        <inertia
-          ixx="${I_sphere}" ixy="0" ixz="0"
-          iyy="${I_sphere}" iyz="0"
-          izz="${I_sphere}"/>
+        <inertia ixx="${I_sphere}" ixy="0" ixz="0"
+                 iyy="${I_sphere}" iyz="0"
+                 izz="${I_sphere}"/>
       </inertial>
     </link>
@@ -39,7 +55,8 @@
       <axis xyz="0 1 0"/>
       <parent link="${prefix}base_link"/>
-      <child link="${prefix}${side}_wheel_link"/>
-      <origin xyz="${x_reflect*wheel_xoff} ${y_reflect*(wheel_separation/2+wheel_yoff)} ${-wheel_radius}" rpy="0 0 0"/>
-      <dynamics damping="0.1" friction="0.0"/>  <!-- 0.1 N·m·s/rad models 520-motor gearbox back-drive resistance -->
+      <child  link="${prefix}${side}_wheel_link"/>
+      <origin xyz="${x_reflect*wheel_xoff} ${y_reflect*(wheel_separation/2+wheel_yoff)} ${-wheel_radius}"
+              rpy="0 0 0"/>
+      <dynamics damping="0.1" friction="0.0"/>
     </joint>
     <gazebo reference="${prefix}${side}_wheel_link">
@@ -47,20 +64,21 @@
         <friction>
           <ode>
-              <mu>1.0</mu>
-              <!-- mu2=0.0: roller axis is free (no friction perpendicular to fdir1).
-                   gz:expressed_in keeps fdir1 in the robot body frame so the LCP
-                   always has a well-defined primary direction even with mu2=0. -->
-              <mu2>0.0</mu2>
-              <!-- gz:expressed_in="base_link" locks fdir1 to the chassis frame.
-                   Without this the vector is in world frame and drifts after rotation.
-                   With it DART correctly applies fdir1 relative to the robot body. -->
-              <fdir1 gz:expressed_in="${prefix}base_link">${fdir1}</fdir1>
+            <!-- High friction along fdir1 (roller grip axis) -->
+            <mu>1.0</mu>
+            <!-- Zero friction perpendicular (roller free-rolling direction) -->
+            <mu2>0.0</mu2>
+            <!-- ignition:expressed_in locks fdir1 to the chassis frame.
+                 base_footprint is the root free-body of the URDF (parent of all wheels),
+                 equivalent to "chassis" in the official Gazebo mecanum demo which uses
+                 expressed_in="chassis". DART requires the canonical root body. -->
+            <fdir1 ignition:expressed_in="${prefix}base_footprint">${fdir1}</fdir1>
+            <slip1>0.0</slip1>
+            <!-- slip2=1: roller rolling direction compliance (1 m/s slip per Newton) -->
+            <slip2>1.0</slip2>
           </ode>
         </friction>
         <contact>
           <ode>
-            <!-- Softer contact (was 1e6) reduces oscillations for 50g wheels -->
             <kp>200000.0</kp>
-            <!-- kd/kp ≈ 0.01 prevents bounce -->
             <kd>2000.0</kd>
             <min_depth>0.001</min_depth>
@@ -69,12 +87,12 @@
       </surface>
       <visual>
-          <material>
-              <ambient>0.2 0.2 0.2 1.0</ambient>
-              <diffuse>0.2 0.2 0.2 1.0</diffuse>
-              <specular>0.2 0.2 0.2 1.0</specular>
-              <emissive>0.0 0.0 0.0 0.0</emissive>
-          </material>
+        <material>
+          <ambient>0.2 0.2 0.2 1.0</ambient>
+          <diffuse>0.2 0.2 0.2 1.0</diffuse>
+          <specular>0.2 0.2 0.2 1.0</specular>
+          <emissive>0.0 0.0 0.0 0.0</emissive>
+        </material>
       </visual>
-  </gazebo>
+    </gazebo>
   </xacro:macro>
 </robot>

File: yahboom_rosmaster_description/urdf/robots/rosmaster_x3.urdf.xacro (robot description, xacro)
@@ -1,4 +1,7 @@
 <?xml version="1.0"?>
-<robot xmlns:xacro="http://www.ros.org/wiki/xacro" xmlns:gz="http://gazebosim.org/schema" name="rosmaster_x3">
+<robot xmlns:xacro="http://www.ros.org/wiki/xacro"
+       xmlns:gz="http://gazebosim.org/schema"
+       xmlns:ignition="http://ignitionrobotics.org/schema"
+       name="rosmaster_x3">
   <xacro:property name="M_PI" value="3.1415926535897931" />
   <xacro:arg name="robot_name" default="rosmaster_x3"/>
@@ -11,7 +14,8 @@
   <xacro:include filename="$(find yahboom_rosmaster_description)/urdf/sensors/imu.urdf.xacro"/>
   <xacro:rosmaster_x3_base prefix="$(arg prefix)"/>
-  <!-- fdir1 defines the roller axis direction (locked to chassis frame via gz:expressed_in).
-       FL/BR diagonal: rollers at -45° to forward  →  (1, -1, 0) normalized
-       FR/BL diagonal: rollers at +45° to forward  →  (1,  1, 0) normalized -->
+  <!-- fdir1 = roller grip direction in base_footprint frame via ignition:expressed_in.
+       Matches the official Gazebo mecanum demo (expressed_in="chassis", same topology).
+       FL/BR: grip along (0.707, -0.707, 0) — "A"-type rollers
+       FR/BL: grip along (0.707,  0.707, 0) — "B"-type rollers -->
   <xacro:mecanum_wheel
     prefix="$(arg prefix)"
@@ -68,15 +72,4 @@
       </plugin>
     </gazebo>
-    <!-- VelocityControl: directly applies world-frame velocity to the robot body,
-         bypassing the DART anisotropic-friction-expressed_in issue.
-         A ROS node (mecanum_velocity_control.py) transforms body-frame /cmd_vel
-         to world-frame before publishing to /cmd_vel_world_frame, which is bridged
-         to this plugin's Ignition topic /cmd_vel_world via ros_gz_bridge. -->
-    <gazebo>
-      <plugin filename="gz-sim-velocity-control-system"
-              name="gz::sim::systems::VelocityControl">
-        <topic>/cmd_vel_world</topic>
-      </plugin>
-    </gazebo>
   </xacro:if>
   <!-- ros2_control joints/interfaces for the robot -->
