Commit message: Fix Gazebo mecanum strafing with native drive
Use the native Fortress MecanumDrive system for wheel commands while keeping gz_ros2_control read-only for joint states. Add a cmd_vel watchdog and wheel-state odometry so /cmd_vel, /odom, and TF keep their ROS-facing contracts without relying on Gazebo ground truth.

Attach anisotropic wheel friction to the wheel collision and express fdir1 in base_footprint with ignition:expressed_in, matching the spawned SDF root body so physical strafing works through wheel-ground contact.

File: yahboom_rosmaster_description/urdf/control/rosmaster_x3_ros2_control.urdf.xacro (robot description, xacro)
@@ -7,20 +7,16 @@
             </hardware>
             <joint name="${prefix}front_left_wheel_joint">
-              <command_interface name="velocity"/>
               <state_interface name="position"/>
               <state_interface name="velocity"/>
             </joint>
             <joint name="${prefix}front_right_wheel_joint">
-              <command_interface name="velocity"/>
               <state_interface name="position"/>
               <state_interface name="velocity"/>
             </joint>
             <joint name="${prefix}back_left_wheel_joint">
-              <command_interface name="velocity"/>
               <state_interface name="position"/>
               <state_interface name="velocity"/>
             </joint>
             <joint name="${prefix}back_right_wheel_joint">
-              <command_interface name="velocity"/>
               <state_interface name="position"/>
               <state_interface name="velocity"/>

File: yahboom_rosmaster_description/urdf/mech/mecanum_wheel.urdf.xacro (robot description, xacro)
@@ -5,13 +5,11 @@
     mu=1.0  along fdir1 (roller grip direction — high friction)
     mu2=0.0 perpendicular to fdir1 (roller free-rolling direction — zero friction)
-  fdir1 is expressed in the robot base_link frame via ignition:expressed_in so
-  the friction direction rotates with the chassis at any heading.
-  With Bullet physics (ignition-physics5-bullet-plugin), expressed_in is
-  re-evaluated every physics step → correct holonomic motion at any heading.
-  With DART, expressed_in is computed once at model load (one-shot bug) → correct
-  strafing at initial yaw=0 only.
+  fdir1 is expressed in the robot base_footprint frame via ignition:expressed_in
+  to match the native Gazebo mecanum demo's chassis-frame friction directions.
+  Locomotion is commanded by the Gazebo MecanumDrive system; this collision and
+  friction model remains the wheel-ground contact model that DART resolves.
   fdir1 values per wheel (set by caller in rosmaster_x3.urdf.xacro):
-    FL, BR: "0.707107 -0.707107 0"
-    FR, BL: "0.707107  0.707107 0"
+    FL, BR: "1 -1 0"
+    FR, BL: "1  1 0"
 -->
 <robot xmlns:xacro="http://www.ros.org/wiki/xacro"
@@ -23,5 +21,5 @@
   <xacro:property name="wheel_xoff"      value="0.08"    />
   <xacro:property name="wheel_yoff"      value="-0.01"   />
-  <xacro:macro name="mecanum_wheel" params="prefix side x_reflect y_reflect fdir1:='0.707107 0 0'">
+  <xacro:macro name="mecanum_wheel" params="prefix side x_reflect y_reflect fdir1:='1 0 0'">
     <link name="${prefix}${side}_wheel_link">
       <visual>
@@ -61,29 +59,29 @@
     </joint>
     <gazebo reference="${prefix}${side}_wheel_link">
-      <surface>
-        <friction>
-          <ode>
-            <!-- High friction along fdir1 (roller grip axis) -->
-            <mu>1.0</mu>
-            <!-- Zero friction perpendicular (roller free-rolling direction) -->
-            <mu2>0.0</mu2>
-            <!-- ignition:expressed_in locks fdir1 to the chassis frame.
-                 base_footprint is the root free-body of the URDF (parent of all wheels),
-                 equivalent to "chassis" in the official Gazebo mecanum demo which uses
-                 expressed_in="chassis". DART requires the canonical root body. -->
-            <fdir1 ignition:expressed_in="${prefix}base_footprint">${fdir1}</fdir1>
-            <slip1>0.0</slip1>
-            <!-- slip2=1: roller rolling direction compliance (1 m/s slip per Newton) -->
-            <slip2>1.0</slip2>
-          </ode>
-        </friction>
-        <contact>
-          <ode>
-            <kp>200000.0</kp>
-            <kd>2000.0</kd>
-            <min_depth>0.001</min_depth>
-          </ode>
-        </contact>
-      </surface>
+      <collision>
+        <surface>
+          <friction>
+            <ode>
+              <!-- High friction along fdir1 (roller grip axis) -->
+              <mu>1.0</mu>
+              <!-- Zero friction perpendicular (roller free-rolling direction) -->
+              <mu2>0.0</mu2>
+              <!-- ignition:expressed_in locks fdir1 to the chassis frame.
+                   base_footprint is the model root frame, equivalent to "chassis"
+                   in the official Gazebo mecanum demo. -->
+              <fdir1 ignition:expressed_in="${prefix}base_footprint">${fdir1}</fdir1>
+              <slip1>0.0</slip1>
+              <slip2>0.0</slip2>
+            </ode>
+          </friction>
+          <contact>
+            <ode>
+              <kp>200000.0</kp>
+              <kd>2000.0</kd>
+              <min_depth>0.001</min_depth>
+            </ode>
+          </contact>
+        </surface>
+      </collision>
       <visual>
         <material>

File: yahboom_rosmaster_description/urdf/robots/rosmaster_x3.urdf.xacro (robot description, xacro)
@@ -16,6 +16,6 @@
   <!-- fdir1 = roller grip direction in base_footprint frame via ignition:expressed_in.
        Matches the official Gazebo mecanum demo (expressed_in="chassis", same topology).
-       FL/BR: grip along (0.707, -0.707, 0) — "A"-type rollers
-       FR/BL: grip along (0.707,  0.707, 0) — "B"-type rollers -->
+       FL/BR: grip along (1, -1, 0) — "A"-type rollers
+       FR/BL: grip along (1,  1, 0) — "B"-type rollers -->
   <xacro:mecanum_wheel
     prefix="$(arg prefix)"
@@ -23,5 +23,5 @@
     x_reflect="1"
     y_reflect="1"
-    fdir1="0.707107 -0.707107 0"/>
+    fdir1="1 -1 0"/>
   <xacro:mecanum_wheel
     prefix="$(arg prefix)"
@@ -29,5 +29,5 @@
     x_reflect="1"
     y_reflect="-1"
-    fdir1="0.707107 0.707107 0"/>
+    fdir1="1 1 0"/>
   <xacro:mecanum_wheel
     prefix="$(arg prefix)"
@@ -35,5 +35,5 @@
     x_reflect="-1"
     y_reflect="1"
-    fdir1="0.707107 0.707107 0"/>
+    fdir1="1 1 0"/>
   <xacro:mecanum_wheel
     prefix="$(arg prefix)"
@@ -41,5 +41,5 @@
     x_reflect="-1"
     y_reflect="-1"
-    fdir1="0.707107 -0.707107 0"/>
+    fdir1="1 -1 0"/>
   <xacro:rgbd_camera
     prefix="$(arg prefix)"
@@ -65,9 +65,22 @@
     update_rate="15.0"
     topic_name="imu/data"/>
-  <!-- Gazebo Fortress ros2_control plugin (gz_ros2_control) -->
+  <!-- Gazebo Fortress simulation plugins. gz_ros2_control is read-only for
+       wheel state; native MecanumDrive owns wheel velocity commands. -->
   <xacro:if value="$(arg use_gazebo)">
     <gazebo>
       <plugin filename="gz_ros2_control-system" name="gz_ros2_control::GazeboSimROS2ControlPlugin">
         <parameters>$(find yahboom_rosmaster_gazebo)/config/ros2_control.yaml</parameters>
+      </plugin>
+      <plugin filename="ignition-gazebo-mecanum-drive-system"
+              name="ignition::gazebo::systems::MecanumDrive">
+        <front_left_joint>$(arg prefix)front_left_wheel_joint</front_left_joint>
+        <front_right_joint>$(arg prefix)front_right_wheel_joint</front_right_joint>
+        <back_left_joint>$(arg prefix)back_left_wheel_joint</back_left_joint>
+        <back_right_joint>$(arg prefix)back_right_wheel_joint</back_right_joint>
+        <wheelbase>0.16</wheelbase>
+        <wheel_separation>0.149</wheel_separation>
+        <wheel_radius>0.0325</wheel_radius>
+        <min_acceleration>-1.0</min_acceleration>
+        <max_acceleration>1.0</max_acceleration>
       </plugin>
     </gazebo>
