Commit message: Restore and validate simulator sensor interfaces

File: yahboom_rosmaster_description/urdf/control/rosmaster_x3_ros2_control.urdf.xacro (robot description, xacro)
@@ -22,4 +22,18 @@
               <state_interface name="velocity"/>
             </joint>
+            <!-- Match the Gazebo IMU entity so gz_ros2_control can expose its
+                 read-only state without trying to command the sensor. -->
+            <sensor name="${prefix}imu_sensor">
+              <state_interface name="orientation.x"/>
+              <state_interface name="orientation.y"/>
+              <state_interface name="orientation.z"/>
+              <state_interface name="orientation.w"/>
+              <state_interface name="angular_velocity.x"/>
+              <state_interface name="angular_velocity.y"/>
+              <state_interface name="angular_velocity.z"/>
+              <state_interface name="linear_acceleration.x"/>
+              <state_interface name="linear_acceleration.y"/>
+              <state_interface name="linear_acceleration.z"/>
+            </sensor>
       </ros2_control>
   </xacro:macro>

File: yahboom_rosmaster_description/urdf/robots/rosmaster_x3.urdf.xacro (robot description, xacro)
@@ -1,5 +1,4 @@
 <?xml version="1.0"?>
 <robot xmlns:xacro="http://www.ros.org/wiki/xacro"
-       xmlns:gz="http://gazebosim.org/schema"
        xmlns:ignition="http://ignitionrobotics.org/schema"
        name="rosmaster_x3">
@@ -66,5 +65,5 @@
     topic_name="imu/data"/>
   <!-- Gazebo Fortress simulation plugins. gz_ros2_control is read-only for
-       wheel state; native MecanumDrive owns wheel velocity commands. -->
+       wheel and IMU state; native MecanumDrive owns wheel velocity commands. -->
   <xacro:if value="$(arg use_gazebo)">
     <gazebo>

File: yahboom_rosmaster_description/urdf/sensors/imu.urdf.xacro (robot description, xacro)
@@ -56,9 +56,11 @@
         </joint>
         <gazebo reference="${prefix}${frame_id}_link">
-            <material>
-                <ambient>${gazebo_material_ambient}</ambient>
-                <diffuse>${gazebo_material_diffuse}</diffuse>
-                <specular>${gazebo_material_specular}</specular>
-            </material>
+            <visual>
+                <material>
+                    <ambient>${gazebo_material_ambient}</ambient>
+                    <diffuse>${gazebo_material_diffuse}</diffuse>
+                    <specular>${gazebo_material_specular}</specular>
+                </material>
+            </visual>
             <!-- Fortress-native IMU sensor. libgazebo_ros_imu_sensor.so is Classic-only
                  and must not be used here. Data flows via ros_gz_bridge (gz.msgs.IMU →

File: yahboom_rosmaster_description/urdf/sensors/lidar.urdf.xacro (robot description, xacro)
@@ -76,9 +76,11 @@
     </joint>
     <gazebo reference="${prefix}${frame_id}">
-      <material>
-        <ambient>${gazebo_material_ambient}</ambient>
-        <diffuse>${gazebo_material_diffuse}</diffuse>
-        <specular>${gazebo_material_specular}</specular>
-      </material>
+      <visual>
+        <material>
+          <ambient>${gazebo_material_ambient}</ambient>
+          <diffuse>${gazebo_material_diffuse}</diffuse>
+          <specular>${gazebo_material_specular}</specular>
+        </material>
+      </visual>
       <!-- Fortress-native GPU LiDAR. type="ray" (CPU LIDAR) is not supported in Fortress;
            type="gpu_lidar" uses the ogre2 render pipeline (enabled in empty.world).
@@ -112,5 +114,7 @@
             <resolution>${range_resolution}</resolution>
           </range>
-          <noise type="gaussian">
+          <!-- SDFormat's lidar schema uses a child element for the noise type. -->
+          <noise>
+            <type>gaussian</type>
             <mean>${noise_mean}</mean>
             <stddev>${noise_stddev}</stddev>

File: yahboom_rosmaster_description/urdf/sensors/rgbd_camera.urdf.xacro (robot description, xacro)
@@ -124,9 +124,10 @@
     </joint>
     <link name="${prefix}${camera_name}_color_optical_frame"/>
-    <!-- Fortress sensor: uses the gz-sim Sensors system (loaded in the world SDF).
-         Data is bridged to ROS via ros_gz_bridge + ros_gz_image_bridge.
-         libgazebo_ros_camera.so is Classic-only and must NOT be used in Fortress. -->
+    <!-- Fortress RGB-D sensor: publishes <topic>/image, <topic>/depth_image,
+         <topic>/camera_info, and <topic>/points through the Sensors system loaded
+         by the world. Data is bridged to ROS by ros_gz_bridge and ros_gz_image.
+         libgazebo_ros_camera.so is Classic-only and must NOT be used here. -->
     <gazebo reference="${prefix}${camera_name}_link">
-      <sensor name="${prefix}${camera_name}" type="depth_camera">
+      <sensor name="${prefix}${camera_name}" type="rgbd_camera">
         <camera>
           <horizontal_fov>${horizontal_fov}</horizontal_fov>
