Commit message: Add a Gazebo Classic backend so macOS gets LiDAR, SLAM and Nav2
Gazebo Fortress on macOS can neither open its GUI nor run a rendering sensor, so
the Fortress backend leaves Mac users with no Gazebo window and no /scan, which
rules out SLAM and Nav2. Gazebo Classic opens its GUI normally and its CPU
raycast lidar needs no rendering at all, so it can do both. Add it as a second
backend selected by a sim_backend xacro argument and a separate pixi
environment; the Fortress path is untouched and stays the default.

Four defects had to be fixed to make the robot move, each silent in its own way:

- gazebo_ros' own gzserver.launch.py names its system plugins with a hardcoded
  ".so" while a macOS build installs ".dylib", so gzserver came up without
  libgazebo_ros_factory and /spawn_entity never appeared. Start gzserver
  directly with the right suffix instead.
- base_footprint is the URDF root and so the model's canonical link, but it had
  no inertial. Gazebo Classic builds no physics body for a massless link, so
  Model::WorldLinearVel() returned NaN and planar_move could never move the
  robot. Give it a token inertia on this backend.
- planar_move imposes an angular velocity on every link, which contradicts a
  revolute wheel free to spin about its own axis; the ODE solver diverged to
  NaN. Weld the wheels on this backend. They no longer rotate visually, which is
  the main cost of the approach.
- The mecanum roller model pairs mu2=0 with a directional fdir1, leaving ODE a
  degenerate friction pyramid. Classic uses plain isotropic friction, which it
  can afford because planar_move does not rely on wheel grip.

Verified on an M4 Max: drives 0.579 m in 2 s at 0.3 m/s, strafes the same
distance sideways with no forward drift, LiDAR reads 2.925 m to a wall at
2.95 m, slam_toolbox grows the map from 278 to 691 occupied cells, and Nav2
reaches a goal 2 m away to within 0.01 m.

The RGB-D camera stays unavailable: macOS renders it blank on both backends.

Co-Authored-By: Claude Opus 5 (1M context) <noreply@anthropic.com>
Claude-Session: https://claude.ai/code/session_01EdVYHU8DgpEjDU7fB4CNqR

File: yahboom_rosmaster_description/urdf/mech/mecanum_wheel.urdf.xacro (robot description, xacro)
@@ -31,5 +31,7 @@
     mu2:=0.0
     slip1:=0.0
-    slip2:=0.0">
+    slip2:=0.0
+    simple_friction:=false
+    joint_type:=continuous">
     <link name="${prefix}${side}_wheel_link">
       <visual>
@@ -60,5 +62,11 @@
       </inertial>
     </link>
-    <joint name="${prefix}${side}_wheel_joint" type="continuous">
+    <!-- Gazebo Classic drives the base with planar_move, which forces an
+         angular velocity onto every link. A revolute wheel must be free to
+         spin about its own axis, so that command contradicts the joint and
+         the ODE solver diverges to NaN, leaving the robot immobile. Welding
+         the wheels makes the base a single rigid body and planar_move works.
+         Fortress keeps them continuous: MecanumDrive spins them properly. -->
+    <joint name="${prefix}${side}_wheel_joint" type="${joint_type}">
       <axis xyz="0 1 0"/>
       <parent link="${prefix}base_link"/>
@@ -73,14 +81,26 @@
           <friction>
             <ode>
-              <!-- High friction along fdir1 (roller grip axis) -->
-              <mu>${mu}</mu>
-              <!-- Zero friction perpendicular (roller free-rolling direction) -->
-              <mu2>${mu2}</mu2>
-              <!-- ignition:expressed_in locks fdir1 to the chassis frame.
-                   base_footprint is the model root frame, equivalent to "chassis"
-                   in the official Gazebo mecanum demo. -->
-              <fdir1 ignition:expressed_in="${prefix}base_footprint">${fdir1}</fdir1>
-              <slip1>${slip1}</slip1>
-              <slip2>${slip2}</slip2>
+              <xacro:unless value="${simple_friction}">
+                <!-- High friction along fdir1 (roller grip axis) -->
+                <mu>${mu}</mu>
+                <!-- Zero friction perpendicular (roller free-rolling direction) -->
+                <mu2>${mu2}</mu2>
+                <!-- ignition:expressed_in locks fdir1 to the chassis frame.
+                     base_footprint is the model root frame, equivalent to "chassis"
+                     in the official Gazebo mecanum demo. -->
+                <fdir1 ignition:expressed_in="${prefix}base_footprint">${fdir1}</fdir1>
+                <slip1>${slip1}</slip1>
+                <slip2>${slip2}</slip2>
+              </xacro:unless>
+              <!-- Gazebo Classic. The roller model above pairs mu2=0 with a
+                   directional fdir1, which leaves ODE a degenerate friction
+                   pyramid: the moment planar_move drives the body, the solver
+                   returns NaN velocities and the robot never moves. Classic gets
+                   plain low isotropic friction instead; planar_move imposes the
+                   body velocity directly, so it does not rely on wheel grip. -->
+              <xacro:if value="${simple_friction}">
+                <mu>0.1</mu>
+                <mu2>0.1</mu2>
+              </xacro:if>
             </ode>
           </friction>

File: yahboom_rosmaster_description/urdf/mech/rosmaster_x3_base.urdf.xacro (robot description, xacro)
@@ -12,6 +12,20 @@
 <xacro:property name="base_size_z" value="${total_height - (2 * wheel_radius)}" />
 <xacro:property name="base_mass" value="1.5" />  <!-- Real X3: ~1.3 kg chassis+motors+PCBs + ~0.2 kg SBC/mount. Old value 4.6 kg was ~3× too heavy. -->
-<xacro:macro name="rosmaster_x3_base" params="prefix">
-  <link name="${prefix}base_footprint"/>
+<xacro:macro name="rosmaster_x3_base" params="prefix footprint_inertial:=false">
+  <!-- base_footprint is the URDF root and therefore the model's canonical link.
+       Gazebo Classic builds no physics body for a massless link, so queries like
+       Model::WorldLinearVel() return NaN and gazebo_ros_planar_move can never
+       move the robot. A token inertia gives it a body; the mass is four orders
+       of magnitude below the chassis, so dynamics are unaffected. Fortress does
+       not need this and leaves the link empty. -->
+  <link name="${prefix}base_footprint">
+    <xacro:if value="${footprint_inertial}">
+      <inertial>
+        <mass value="0.001"/>
+        <origin xyz="0 0 0" rpy="0 0 0"/>
+        <inertia ixx="1e-6" ixy="0.0" ixz="0.0" iyy="1e-6" iyz="0.0" izz="1e-6"/>
+      </inertial>
+    </xacro:if>
+  </link>
   <link name="${prefix}base_link">
     <visual>

File: yahboom_rosmaster_description/urdf/robots/rosmaster_x3.urdf.xacro (robot description, xacro)
@@ -17,4 +17,11 @@
        Gazebo instead and skip ros2_control entirely. -->
   <xacro:arg name="use_ros2_control" default="true"/>
+  <!-- Which simulator the Gazebo tags target. "fortress" is the upstream
+       backend. "classic" is for macOS, where Fortress cannot render sensors or
+       open its GUI; Gazebo Classic can, and its CPU raycast lidar works there. -->
+  <xacro:arg name="sim_backend" default="fortress"/>
+  <xacro:property name="backend" value="$(arg sim_backend)"/>
+  <!-- Gazebo Classic plugin suffix: conda installs .dylib on macOS, .so on Linux. -->
+  <xacro:arg name="plugin_ext" default=".so"/>
   <!-- Contact parameters are supplied by the simulator motion profile. These
        defaults preserve the ideal description when xacro is expanded directly. -->
@@ -31,5 +38,7 @@
   <xacro:include filename="$(find yahboom_rosmaster_description)/urdf/sensors/lidar.urdf.xacro"/>
   <xacro:include filename="$(find yahboom_rosmaster_description)/urdf/sensors/imu.urdf.xacro"/>
-  <xacro:rosmaster_x3_base prefix="$(arg prefix)"/>
+  <xacro:rosmaster_x3_base
+    prefix="$(arg prefix)"
+    footprint_inertial="${backend == 'classic'}"/>
   <!-- fdir1 = roller grip direction in base_footprint frame via ignition:expressed_in.
        Matches the official Gazebo mecanum demo (expressed_in="chassis", same topology).
@@ -45,5 +54,7 @@
     mu2="$(arg wheel_mu2)"
     slip1="$(arg front_left_slip1)"
-    slip2="$(arg wheel_slip2)"/>
+    slip2="$(arg wheel_slip2)"
+    simple_friction="${backend == 'classic'}"
+    joint_type="${'fixed' if backend == 'classic' else 'continuous'}"/>
   <xacro:mecanum_wheel
     prefix="$(arg prefix)"
@@ -55,5 +66,7 @@
     mu2="$(arg wheel_mu2)"
     slip1="$(arg front_right_slip1)"
-    slip2="$(arg wheel_slip2)"/>
+    slip2="$(arg wheel_slip2)"
+    simple_friction="${backend == 'classic'}"
+    joint_type="${'fixed' if backend == 'classic' else 'continuous'}"/>
   <xacro:mecanum_wheel
     prefix="$(arg prefix)"
@@ -65,5 +78,7 @@
     mu2="$(arg wheel_mu2)"
     slip1="$(arg back_left_slip1)"
-    slip2="$(arg wheel_slip2)"/>
+    slip2="$(arg wheel_slip2)"
+    simple_friction="${backend == 'classic'}"
+    joint_type="${'fixed' if backend == 'classic' else 'continuous'}"/>
   <xacro:mecanum_wheel
     prefix="$(arg prefix)"
@@ -75,5 +90,7 @@
     mu2="$(arg wheel_mu2)"
     slip1="$(arg back_right_slip1)"
-    slip2="$(arg wheel_slip2)"/>
+    slip2="$(arg wheel_slip2)"
+    simple_friction="${backend == 'classic'}"
+    joint_type="${'fixed' if backend == 'classic' else 'continuous'}"/>
   <xacro:rgbd_camera
     prefix="$(arg prefix)"
@@ -81,5 +98,5 @@
     xyz_offset="0.105 0 0.05"
     rpy_offset="0 0 0"
-    enable_gz_sensor="$(arg render_sensors)"/>
+    enable_gz_sensor="${backend == 'fortress' and '$(arg render_sensors)' in ['true', 'True', '1']}"/>
   <xacro:lidar_sensor
     prefix="$(arg prefix)"
@@ -92,5 +109,7 @@
     update_rate="5"
     topic_name="scan"
-    enable_gz_sensor="$(arg render_sensors)"/>
+    enable_gz_sensor="${backend == 'fortress' and '$(arg render_sensors)' in ['true', 'True', '1']}"
+    classic_sensor="${backend == 'classic'}"
+    plugin_ext="$(arg plugin_ext)"/>
   <xacro:imu_sensor
     prefix="$(arg prefix)"
@@ -103,5 +122,32 @@
   <!-- Gazebo Fortress simulation plugins. gz_ros2_control is read-only for
        wheel and IMU state; native MecanumDrive owns wheel velocity commands. -->
-  <xacro:if value="$(arg use_gazebo)">
+  <xacro:if value="${backend == 'classic'}">
+    <gazebo>
+      <!-- ODE parks resting bodies, and a parked body ignores the velocity
+           planar_move sets, so the robot never starts moving. -->
+      <allow_auto_disable>false</allow_auto_disable>
+      <!-- Holonomic base drive. planar_move consumes linear.x, linear.y and
+           angular.z, so it reproduces mecanum strafing, and it owns both /odom
+           and the odom->base_footprint transform. -->
+      <plugin name="planar_move" filename="libgazebo_ros_planar_move$(arg plugin_ext)">
+        <ros>
+          <remapping>cmd_vel:=cmd_vel</remapping>
+          <remapping>odom:=odom</remapping>
+        </ros>
+        <update_rate>50</update_rate>
+        <publish_odom>true</publish_odom>
+        <publish_odom_tf>true</publish_odom_tf>
+        <odometry_frame>odom</odometry_frame>
+        <robot_base_frame>$(arg prefix)base_footprint</robot_base_frame>
+        <covariance_x>0.0001</covariance_x>
+        <covariance_y>0.0001</covariance_y>
+        <covariance_yaw>0.01</covariance_yaw>
+      </plugin>
+      <!-- No joint state publisher here: the wheels are welded on this backend,
+           so there is nothing to report and robot_state_publisher emits their
+           transforms on /tf_static instead. -->
+    </gazebo>
+  </xacro:if>
+  <xacro:if value="${backend == 'fortress' and '$(arg use_gazebo)' in ['true', 'True', '1']}">
     <gazebo>
       <xacro:if value="$(arg use_ros2_control)">

File: yahboom_rosmaster_description/urdf/sensors/lidar.urdf.xacro (robot description, xacro)
@@ -37,5 +37,7 @@
     visualize:=false
     enable_collision:=false
-    enable_gz_sensor:=true">
+    enable_gz_sensor:=true
+    classic_sensor:=false
+    plugin_ext:=.so">
     <xacro:property name="radius" value="${lidar_width/2}" />
     <xacro:property name="ixx_iyy" value="${(mass/12) * (3 * radius * radius + lidar_height * lidar_height)}" />
@@ -129,4 +131,43 @@
       </sensor>
       </xacro:if>
+      <!-- Gazebo Classic. type="ray" is the CPU raycast lidar: it queries the
+           physics engine instead of the render pipeline, so unlike gpu_lidar it
+           produces correct ranges on macOS, where server-side rendering is
+           broken. -->
+      <xacro:if value="${classic_sensor}">
+        <sensor name="${prefix}lidar_sensor" type="ray">
+          <pose>0 0 0 0 0 0</pose>
+          <always_on>${always_on}</always_on>
+          <visualize>${visualize}</visualize>
+          <update_rate>${update_rate}</update_rate>
+          <ray>
+            <scan>
+              <horizontal>
+                <samples>${ray_count}</samples>
+                <resolution>1</resolution>
+                <min_angle>${min_angle}</min_angle>
+                <max_angle>${max_angle}</max_angle>
+              </horizontal>
+            </scan>
+            <range>
+              <min>${min_range}</min>
+              <max>${max_range}</max>
+              <resolution>${range_resolution}</resolution>
+            </range>
+            <noise>
+              <type>gaussian</type>
+              <mean>${noise_mean}</mean>
+              <stddev>${noise_stddev}</stddev>
+            </noise>
+          </ray>
+          <plugin name="${prefix}lidar_controller" filename="libgazebo_ros_ray_sensor${plugin_ext}">
+            <ros>
+              <remapping>~/out:=${topic_name}</remapping>
+            </ros>
+            <output_type>sensor_msgs/LaserScan</output_type>
+            <frame_name>${prefix}${frame_id}</frame_name>
+          </plugin>
+        </sensor>
+      </xacro:if>
     </gazebo>
   </xacro:macro>
