Commit message: Add ground truth and stress motion profiles

File: yahboom_rosmaster_description/urdf/mech/mecanum_wheel.urdf.xacro (robot description, xacro)
@@ -2,7 +2,8 @@
 <!--
   Mecanum wheel with sphere collision + fdir1 anisotropic friction.
-  Each wheel is a sphere (single contact point) with:
-    mu=1.0  along fdir1 (roller grip direction — high friction)
-    mu2=0.0 perpendicular to fdir1 (roller free-rolling direction — zero friction)
+  Each wheel is a sphere (single contact point) with profile-selected contact
+  values. The ideal profile uses mu=1.0 along fdir1 and mu2=0.0 perpendicular
+  to fdir1; the default stress profile adds deterministic compliance, roller
+  resistance, and per-wheel asymmetry.
   fdir1 is expressed in the robot base_footprint frame via ignition:expressed_in
   to match the native Gazebo mecanum demo's chassis-frame friction directions.
@@ -21,5 +22,14 @@
   <xacro:property name="wheel_xoff"      value="0.08"    />
   <xacro:property name="wheel_yoff"      value="-0.01"   />
-  <xacro:macro name="mecanum_wheel" params="prefix side x_reflect y_reflect fdir1:='1 0 0'">
+  <xacro:macro name="mecanum_wheel" params="
+    prefix
+    side
+    x_reflect
+    y_reflect
+    fdir1:='1 0 0'
+    mu:=1.0
+    mu2:=0.0
+    slip1:=0.0
+    slip2:=0.0">
     <link name="${prefix}${side}_wheel_link">
       <visual>
@@ -64,13 +74,13 @@
             <ode>
               <!-- High friction along fdir1 (roller grip axis) -->
-              <mu>1.0</mu>
+              <mu>${mu}</mu>
               <!-- Zero friction perpendicular (roller free-rolling direction) -->
-              <mu2>0.0</mu2>
+              <mu2>${mu2}</mu2>
               <!-- ignition:expressed_in locks fdir1 to the chassis frame.
                    base_footprint is the model root frame, equivalent to "chassis"
                    in the official Gazebo mecanum demo. -->
               <fdir1 ignition:expressed_in="${prefix}base_footprint">${fdir1}</fdir1>
-              <slip1>0.0</slip1>
-              <slip2>0.0</slip2>
+              <slip1>${slip1}</slip1>
+              <slip2>${slip2}</slip2>
             </ode>
           </friction>

File: yahboom_rosmaster_description/urdf/robots/rosmaster_x3.urdf.xacro (robot description, xacro)
@@ -7,4 +7,13 @@
   <xacro:arg name="prefix" default=""/>
   <xacro:arg name="use_gazebo" default="false"/>
+  <!-- Contact parameters are supplied by the simulator motion profile. These
+       defaults preserve the ideal description when xacro is expanded directly. -->
+  <xacro:arg name="wheel_mu" default="1.0"/>
+  <xacro:arg name="wheel_mu2" default="0.0"/>
+  <xacro:arg name="wheel_slip2" default="0.0"/>
+  <xacro:arg name="front_left_slip1" default="0.0"/>
+  <xacro:arg name="front_right_slip1" default="0.0"/>
+  <xacro:arg name="back_left_slip1" default="0.0"/>
+  <xacro:arg name="back_right_slip1" default="0.0"/>
   <xacro:include filename="$(find yahboom_rosmaster_description)/urdf/mech/rosmaster_x3_base.urdf.xacro"/>
   <xacro:include filename="$(find yahboom_rosmaster_description)/urdf/mech/mecanum_wheel.urdf.xacro"/>
@@ -22,5 +31,9 @@
     x_reflect="1"
     y_reflect="1"
-    fdir1="1 -1 0"/>
+    fdir1="1 -1 0"
+    mu="$(arg wheel_mu)"
+    mu2="$(arg wheel_mu2)"
+    slip1="$(arg front_left_slip1)"
+    slip2="$(arg wheel_slip2)"/>
   <xacro:mecanum_wheel
     prefix="$(arg prefix)"
@@ -28,5 +41,9 @@
     x_reflect="1"
     y_reflect="-1"
-    fdir1="1 1 0"/>
+    fdir1="1 1 0"
+    mu="$(arg wheel_mu)"
+    mu2="$(arg wheel_mu2)"
+    slip1="$(arg front_right_slip1)"
+    slip2="$(arg wheel_slip2)"/>
   <xacro:mecanum_wheel
     prefix="$(arg prefix)"
@@ -34,5 +51,9 @@
     x_reflect="-1"
     y_reflect="1"
-    fdir1="1 1 0"/>
+    fdir1="1 1 0"
+    mu="$(arg wheel_mu)"
+    mu2="$(arg wheel_mu2)"
+    slip1="$(arg back_left_slip1)"
+    slip2="$(arg wheel_slip2)"/>
   <xacro:mecanum_wheel
     prefix="$(arg prefix)"
@@ -40,5 +61,9 @@
     x_reflect="-1"
     y_reflect="-1"
-    fdir1="1 -1 0"/>
+    fdir1="1 -1 0"
+    mu="$(arg wheel_mu)"
+    mu2="$(arg wheel_mu2)"
+    slip1="$(arg back_right_slip1)"
+    slip2="$(arg wheel_slip2)"/>
   <xacro:rgbd_camera
     prefix="$(arg prefix)"
@@ -83,4 +108,16 @@
         <max_acceleration>1.0</max_acceleration>
       </plugin>
+      <!-- Measurement-only world pose. It is bridged to /ground_truth/odom but
+           its Pose_V output is intentionally not bridged into the ROS TF tree. -->
+      <plugin filename="ignition-gazebo-odometry-publisher-system"
+              name="ignition::gazebo::systems::OdometryPublisher">
+        <odom_frame>world</odom_frame>
+        <robot_base_frame>$(arg prefix)base_footprint</robot_base_frame>
+        <dimensions>3</dimensions>
+        <odom_publish_frequency>50</odom_publish_frequency>
+        <odom_topic>/model/rosmaster_x3/ground_truth</odom_topic>
+        <odom_covariance_topic>/model/rosmaster_x3/ground_truth_with_covariance</odom_covariance_topic>
+        <tf_topic>/model/rosmaster_x3/ground_truth_pose</tf_topic>
+      </plugin>
     </gazebo>
   </xacro:if>

Commit message: Add Donatello CAD visuals and simulator documentation

File: yahboom_rosmaster_description/urdf/mech/mecanum_wheel.urdf.xacro (robot description, xacro)
@@ -36,11 +36,11 @@
     <link name="${prefix}${side}_wheel_link">
       <visual>
-        <origin xyz="0 0 0" rpy="${pi/2} 0 0"/>
+        <!-- Keep the established joint and collision position. Moving the
+             visual 10 mm along its rotation axis matches the assembled CAD
+             without changing contact geometry or drivetrain behavior. -->
+        <origin xyz="0 ${-y_reflect*wheel_yoff} 0" rpy="0 0 0"/>
         <geometry>
-          <mesh filename="file://$(find yahboom_rosmaster_description)/meshes/rosmaster_x3/visual/${side}_wheel_X3.STL"/>
+          <mesh filename="file://$(find yahboom_rosmaster_description)/meshes/rosmaster_x3/cad_visual/${side}_wheel.obj"/>
         </geometry>
-        <material name="dark_gray">
-          <color rgba="0.2 0.2 0.2 1.0"/>
-        </material>
       </visual>
       <!-- Sphere gives a single contact point. Required for ignition:expressed_in
@@ -114,12 +114,4 @@
         </surface>
       </collision>
-      <visual>
-        <material>
-          <ambient>0.2 0.2 0.2 1.0</ambient>
-          <diffuse>0.2 0.2 0.2 1.0</diffuse>
-          <specular>0.2 0.2 0.2 1.0</specular>
-          <emissive>0.0 0.0 0.0 0.0</emissive>
-        </material>
-      </visual>
     </gazebo>
   </xacro:macro>

File: yahboom_rosmaster_description/urdf/mech/rosmaster_x3_base.urdf.xacro (robot description, xacro)
@@ -31,9 +31,6 @@
     <visual>
         <geometry>
-            <mesh filename="file://$(find yahboom_rosmaster_description)/meshes/rosmaster_x3/visual/base_link_X3.STL"/>
+            <mesh filename="file://$(find yahboom_rosmaster_description)/meshes/rosmaster_x3/cad_visual/rosmaster_base.obj"/>
         </geometry>
-        <material name="green">
-          <color rgba="0 0.7 0 1"/>
-        </material>
         <origin xyz="0 0 0" rpy="0 0 0"/>
     </visual>
@@ -53,13 +50,4 @@
     </inertial>
   </link>
-  <gazebo reference="${prefix}base_link">
-    <visual>
-        <material>
-            <ambient>0 0.7 0 1</ambient>
-            <diffuse>0 0.7 0 1</diffuse>
-            <specular>0 0.7 0 1</specular>
-        </material>
-    </visual>
-  </gazebo>
   <joint name="${prefix}base_joint" type="fixed">
     <parent link="${prefix}base_footprint"/>

File: yahboom_rosmaster_description/urdf/robots/rosmaster_x3.urdf.xacro (robot description, xacro)
@@ -118,6 +118,4 @@
     rpy_offset="0 0 ${M_PI}"
     min_range="${0.25 if backend == 'classic' else 0.05}"
-    mesh_xyz_offset="0 0 0"
-    mesh_rpy_offset="${-M_PI/2} 0 0"
     update_rate="5"
     topic_name="scan"

File: yahboom_rosmaster_description/urdf/sensors/lidar.urdf.xacro (robot description, xacro)
@@ -6,10 +6,10 @@
     parent:='base_link'
     frame_id:='laser_link'
-    mesh_file:='file://$(find yahboom_rosmaster_description)/meshes/rplidar/rplidar_s2.stl'
+    mesh_file:='file://$(find yahboom_rosmaster_description)/meshes/rosmaster_x3/cad_visual/lidar.obj'
     xyz_offset:='0.043 0 0.110'
     rpy_offset:='0 0 ${M_PI}'
     mesh_xyz_offset:='0 0 0'
-    mesh_rpy_offset:='${-M_PI/2} 0 0'
-    mesh_scale:='0.001 0.001 0.001'
+    mesh_rpy_offset:='0 0 0'
+    mesh_scale:='1 1 1'
     collision_xyz_offset:='0 0 0'
     collision_rpy_offset:='0 0 0'
@@ -19,9 +19,4 @@
     lidar_height:=0.0398
     mass:=0.185
-    material_name:='rplidar_black'
-    material_color:='0.1 0.1 0.1 1'
-    gazebo_material_ambient:='0.1 0.1 0.1 1'
-    gazebo_material_diffuse:='0.1 0.1 0.1 1'
-    gazebo_material_specular:='0.1 0.1 0.1 1'
     update_rate:=10
     ray_count:=1080
@@ -44,4 +39,10 @@
     <xacro:property name="izz" value="${(mass/2) * (radius * radius)}" />
     <link name="${prefix}${frame_id}">
+      <visual>
+        <origin xyz="${mesh_xyz_offset}" rpy="${mesh_rpy_offset}"/>
+        <geometry>
+          <mesh filename="${mesh_file}" scale="${mesh_scale}"/>
+        </geometry>
+      </visual>
       <xacro:if value="${enable_collision}">
         <collision>
@@ -70,10 +71,9 @@
     </joint>
     <gazebo reference="${prefix}${frame_id}">
+      <!-- The detailed CAD housing encloses the GPU ray origin. Give only this
+           visual a private render bit so the LiDAR can ignore its own shell
+           without hiding the chassis, wheels, or camera from sensors. -->
       <visual>
-        <material>
-          <ambient>${gazebo_material_ambient}</ambient>
-          <diffuse>${gazebo_material_diffuse}</diffuse>
-          <specular>${gazebo_material_specular}</specular>
-        </material>
+        <visibility_flags>1</visibility_flags>
       </visual>
       <!-- Fortress-native GPU LiDAR. type="ray" (CPU LIDAR) is not supported in Fortress;
@@ -94,4 +94,5 @@
         <gz_frame_id>${prefix}${frame_id}</gz_frame_id>
         <lidar>
+          <visibility_mask>4294967294</visibility_mask>
           <scan>
             <horizontal>

File: yahboom_rosmaster_description/urdf/sensors/rgbd_camera.urdf.xacro (robot description, xacro)
@@ -6,9 +6,9 @@
     camera_name:='cam_1'
     parent:='base_link'
-    mesh_file:='file://$(find yahboom_rosmaster_description)/meshes/intel_realsense/visual/d435.stl'
+    mesh_file:='file://$(find yahboom_rosmaster_description)/meshes/rosmaster_x3/cad_visual/camera.obj'
     xyz_offset:='0.105 0 0.05'
     rpy_offset:='0 -0.50 0'
     mesh_xyz_offset:='0 0 0'
-    mesh_rpy_offset:='${M_PI/2} 0.0 ${M_PI/2}'
+    mesh_rpy_offset:='0 0 0'
     collision_xyz_offset:='0 0 0'
     collision_rpy_offset:='0 0 0'
@@ -35,6 +35,4 @@
     iyz:=0.0
     izz:=0.003879257
-    material_name:='aluminum'
-    material_color:='0.5 0.5 0.5 1'
     horizontal_fov:=1.5184
     image_width:=424
@@ -42,5 +40,5 @@
     clip_near:=0.05
     clip_far:=8.0
-    update_rate:=2
+    update_rate:=5
     always_on:=1
     visualize:=false
@@ -61,7 +59,4 @@
           <mesh filename="${mesh_file}" />
         </geometry>
-        <material name="${material_name}">
-          <color rgba="${material_color}"/>
-        </material>
       </visual>
       <xacro:if value="${enable_collision}">

Commit message: Correct wheel geometry and ground truth alignment

File: yahboom_rosmaster_description/urdf/mech/mecanum_wheel.urdf.xacro (robot description, xacro)
@@ -21,5 +21,4 @@
   <xacro:property name="wheel_mass"      value="0.05"    />
   <xacro:property name="wheel_xoff"      value="0.08"    />
-  <xacro:property name="wheel_yoff"      value="-0.01"   />
   <xacro:macro name="mecanum_wheel" params="
     prefix
@@ -36,8 +35,7 @@
     <link name="${prefix}${side}_wheel_link">
       <visual>
-        <!-- Keep the established joint and collision position. Moving the
-             visual 10 mm along its rotation axis matches the assembled CAD
-             without changing contact geometry or drivetrain behavior. -->
-        <origin xyz="0 ${-y_reflect*wheel_yoff} 0" rpy="0 0 0"/>
+        <!-- The generated mesh is link-local; no additional visual offset is
+             needed once the joint uses the measured lateral wheel centre. -->
+        <origin xyz="0 0 0" rpy="0 0 0"/>
         <geometry>
           <mesh filename="file://$(find yahboom_rosmaster_description)/meshes/rosmaster_x3/cad_visual/${side}_wheel.obj"/>
@@ -72,5 +70,5 @@
       <parent link="${prefix}base_link"/>
       <child  link="${prefix}${side}_wheel_link"/>
-      <origin xyz="${x_reflect*wheel_xoff} ${y_reflect*(wheel_separation/2+wheel_yoff)} ${-wheel_radius}"
+      <origin xyz="${x_reflect*wheel_xoff} ${y_reflect*wheel_separation/2} ${-wheel_radius}"
               rpy="0 0 0"/>
       <dynamics damping="0.1" friction="0.0"/>

Commit message: fix(description): put base_footprint on the floor at physical height
base_footprint sat at wheel-axle height (32.5 mm up) and base_link at
65 mm, while the physical X3 has base_footprint on the floor and
base_link 71.4 mm up with the axles 38.9 mm below it
(physical_rosmaster yahboomcar_X3.urdf.xacro, confirmed by a tape
measurement of the camera height).

Move the wheel joints to the measured axle drop, raise base_joint to
71.4 mm and spawn at z=0 on both backends. The CAD visuals, chassis
collision and inertia were authored with the axles one wheel radius
below base_link, so shift them by the 6.4 mm difference: the rendered
robot and its physics body stay exactly where they were in the world,
and only the frames move. Sensor offsets from base_link are unchanged,
so the LiDAR and IMU now sit at their physical heights.

The description contract gains a check that every wheel touches
base_footprint z=0, and no longer infers the wheel radius from the
axle drop.

Refs #42

File: yahboom_rosmaster_description/urdf/mech/mecanum_wheel.urdf.xacro (robot description, xacro)
@@ -21,4 +21,9 @@
   <xacro:property name="wheel_mass"      value="0.05"    />
   <xacro:property name="wheel_xoff"      value="0.08"    />
+  <!-- Wheel axles sit this far below base_link on the physical X3 (measured on
+       x3-c; physical_rosmaster yahboomcar_X3.urdf.xacro front_wheel_drop), so
+       base_link is 71.4 mm above the floor. The measured rear axles are within
+       0.6 mm of this; one value keeps the four contacts level. -->
+  <xacro:property name="wheel_axle_drop" value="0.0389"  />
   <xacro:macro name="mecanum_wheel" params="
     prefix
@@ -70,5 +75,5 @@
       <parent link="${prefix}base_link"/>
       <child  link="${prefix}${side}_wheel_link"/>
-      <origin xyz="${x_reflect*wheel_xoff} ${y_reflect*wheel_separation/2} ${-wheel_radius}"
+      <origin xyz="${x_reflect*wheel_xoff} ${y_reflect*wheel_separation/2} ${-wheel_axle_drop}"
               rpy="0 0 0"/>
       <dynamics damping="0.1" friction="0.0"/>

File: yahboom_rosmaster_description/urdf/mech/rosmaster_x3_base.urdf.xacro (robot description, xacro)
@@ -12,4 +12,11 @@
 <xacro:property name="base_size_z" value="${total_height - (2 * wheel_radius)}" />
 <xacro:property name="base_mass" value="1.5" />  <!-- Real X3: ~1.3 kg chassis+motors+PCBs + ~0.2 kg SBC/mount. Old value 4.6 kg was ~3× too heavy. -->
+<!-- base_footprint is on the floor and base_link sits wheel_axle_drop
+     (mecanum_wheel.urdf.xacro) above the axles, as on the physical X3. The
+     chassis visual, collision and inertia were authored with base_link one
+     wheel radius above the axles (tools/convert_rosmaster_cad.py), so they
+     are shifted by the difference to keep resting on the wheels. -->
+<xacro:property name="base_link_height" value="${wheel_radius + wheel_axle_drop}" />
+<xacro:property name="chassis_origin_z" value="${wheel_radius - wheel_axle_drop}" />
 <xacro:macro name="rosmaster_x3_base" params="prefix footprint_inertial:=false">
   <!-- base_footprint is the URDF root and therefore the model's canonical link.
@@ -33,5 +40,5 @@
             <mesh filename="file://$(find yahboom_rosmaster_description)/meshes/rosmaster_x3/cad_visual/rosmaster_base.obj"/>
         </geometry>
-        <origin xyz="0 0 0" rpy="0 0 0"/>
+        <origin xyz="0 0 ${chassis_origin_z}" rpy="0 0 0"/>
     </visual>
     <collision>
@@ -39,8 +46,8 @@
             <box size="${base_size_x} ${base_size_y} ${base_size_z}"/>
         </geometry>
-        <origin xyz="${base_x_offset} 0 ${base_size_z/2 + wheel_radius/4}" rpy="0 0 0"/>
+        <origin xyz="${base_x_offset} 0 ${base_size_z/2 + wheel_radius/4 + chassis_origin_z}" rpy="0 0 0"/>
     </collision>
     <inertial>
-        <origin xyz="${base_x_offset} 0 ${base_size_z/2 + wheel_radius/4}" rpy="0 0 0"/>
+        <origin xyz="${base_x_offset} 0 ${base_size_z/2 + wheel_radius/4 + chassis_origin_z}" rpy="0 0 0"/>
         <mass value="${base_mass}"/>
         <inertia
@@ -53,5 +60,5 @@
     <parent link="${prefix}base_footprint"/>
     <child link="${prefix}base_link"/>
-    <origin xyz="0 0 ${wheel_radius}" rpy="0 0 0"/>
+    <origin xyz="0 0 ${base_link_height}" rpy="0 0 0"/>
   </joint>
 </xacro:macro>

File: yahboom_rosmaster_description/urdf/robots/rosmaster_x3.urdf.xacro (robot description, xacro)
@@ -103,8 +103,9 @@
     xyz_offset="0.105 0 0.05"
     rpy_offset="0 0 0"
+    mesh_xyz_offset="0 0 ${chassis_origin_z}"
     enable_gz_sensor="${backend == 'fortress' and '$(arg render_sensors)' in ['true', 'True', '1']}"/>
   <!-- Classic's CPU raycast starts each ray at range_min, so anything nearer is
        skipped rather than clamped. The chassis collision box spans x [-0.181,
-       0.119], y +/-0.069, z [0.008, 0.205] about base_link and so encloses this
+       0.119], y +/-0.069, z [0.002, 0.199] about base_link and so encloses this
        mount, putting its furthest corner 0.2345 m away. Any range_min below
        that starts part of the sweep inside the hull and those beams return the
@@ -117,4 +118,5 @@
     xyz_offset="0.043 0 0.110"
     rpy_offset="0 0 ${M_PI}"
+    mesh_xyz_offset="0 0 ${chassis_origin_z}"
     min_range="${0.25 if backend == 'classic' else 0.05}"
     update_rate="5"
