Commit message: Apple Silicon backend with LiDAR, SLAM and Nav2, plus Tadeo's simulation work integrated (#2)
* Run the simulation natively on Apple Silicon via RoboStack

macOS has no ROS 2 Humble debs, so the environment comes from RoboStack conda
packages pinned in pixi.toml and pixi.lock. Linux behaviour is unchanged: both
new xacro arguments default to true, and every macOS default is selected by a
platform check in the launch file.

Five failures had to be fixed to get there:

- Gazebo seeds its plugin search from LD_LIBRARY_PATH, which conda never sets
  and macOS does not use, so gz_ros2_control-system never loaded.
- A Mac exposes ~20 multicast interfaces. DDS participants picked different
  ones and never discovered each other, so nodes saw a partial ROS graph and
  waited forever on services that were running. Same for Gazebo's transport.
- Activating a controller aborts the server: ros2_control waits on a condition
  variable holding a deferred, unlocked mutex, which libc++ rejects with EPERM
  inside a noexcept function. Gazebo's own JointStatePublisher feeds
  /joint_states through ros_gz_bridge instead.
- QT_QPA_PLATFORM=xcb, a Wayland workaround, breaks every Qt app on macOS.
- RViz's Camera display builds a second render panel and aborts RViz.

Rendering sensors and the Gazebo GUI stay unavailable on macOS. Both initialise
ogre2 off the main thread, which macOS forbids for window creation. The fix
exists only in Garden and newer (gz-sim#960, gz-sim#1225) and cannot be
backported here, since libignition-rendering6 requires ogre-next 2.2.x and no
conda-forge build of that series ships the Metal render system. RViz replaces
the Gazebo GUI, and anything needing /scan must run on Linux.

Verified on an M4 Max: robot spawns and drives 0.594 m in 2 s at 0.3 m/s,
mecanum strafing is clean, and /clock, /joint_states, /odom, /imu/data and /tf
all publish.

Co-Authored-By: Claude Opus 5 (1M context) <noreply@anthropic.com>
Claude-Session: https://claude.ai/code/session_01EdVYHU8DgpEjDU7fB4CNqR

* Record why newer Gazebo is not the macOS escape hatch

Gazebo Harmonic carries the upstream fix for rendering sensors on macOS, so it
is the obvious thing to reach for next. A scratch RoboStack Jazzy environment
confirmed Harmonic 8.10 ships RenderSystem_Metal and starts without the window
error, but the server then hung during world load with no sensors present.
Note the result so the next person does not repeat the experiment.

Co-Authored-By: Claude Opus 5 (1M context) <noreply@anthropic.com>
Claude-Session: https://claude.ai/code/session_01EdVYHU8DgpEjDU7fB4CNqR

* Pace macOS joint state to the rate joint_state_broadcaster uses

Gazebo's JointStatePublisher has no rate control and publishes every sim step,
so /joint_states arrived near 1 kHz instead of the 30 Hz ros2_control gives on
Linux, dragging /odom and /tf up with it. Bridge to /joint_states_raw and
throttle to 30 Hz.

Also name the bridge node: it shared /ros_gz_bridge with the sensor bridge,
which ros2 node list flagged as a duplicate name.

Co-Authored-By: Claude Opus 5 (1M context) <noreply@anthropic.com>
Claude-Session: https://claude.ai/code/session_01EdVYHU8DgpEjDU7fB4CNqR

* Add a Gazebo Classic backend so macOS gets LiDAR, SLAM and Nav2

Gazebo Fortress on macOS can neither open its GUI nor run a rendering sensor, so
the Fortress backend leaves Mac users with no Gazebo window and no /scan, which
rules out SLAM and Nav2. Gazebo Classic opens its GUI normally and its CPU
raycast lidar needs no rendering at all, so it can do both. Add it as a second
backend selected by a sim_backend xacro argument and a separate pixi
environment; the Fortress path is untouched and stays the default.

Four defects had to be fixed to make the robot move, each silent in its own way:

- gazebo_ros' own gzserver.launch.py names its system plugins with a hardcoded
  ".so" while a macOS build installs ".dylib", so gzserver came up without
  libgazebo_ros_factory and /spawn_entity never appeared. Start gzserver
  directly with the right suffix instead.
- base_footprint is the URDF root and so the model's canonical link, but it had
  no inertial. Gazebo Classic builds no physics body for a massless link, so
  Model::WorldLinearVel() returned NaN and planar_move could never move the
  robot. Give it a token inertia on this backend.
- planar_move imposes an angular velocity on every link, which contradicts a
  revolute wheel free to spin about its own axis; the ODE solver diverged to
  NaN. Weld the wheels on this backend. They no longer rotate visually, which is
  the main cost of the approach.
- The mecanum roller model pairs mu2=0 with a directional fdir1, leaving ODE a
  degenerate friction pyramid. Classic uses plain isotropic friction, which it
  can afford because planar_move does not rely on wheel grip.

Verified on an M4 Max: drives 0.579 m in 2 s at 0.3 m/s, strafes the same
distance sideways with no forward drift, LiDAR reads 2.925 m to a wall at
2.95 m, slam_toolbox grows the map from 278 to 691 occupied cells, and Nav2
reaches a goal 2 m away to within 0.01 m.

The RGB-D camera stays unavailable: macOS renders it blank on both backends.

Co-Authored-By: Claude Opus 5 (1M context) <noreply@anthropic.com>
Claude-Session: https://claude.ai/code/session_01EdVYHU8DgpEjDU7fB4CNqR

* Keep the Fortress task names unambiguous

The classic environment reused build/sim/stop/clean, so pixi refused to run them
without --environment and the documented `pixi run sim` broke. Give the classic
tasks distinct names; pixi then resolves each to the right environment on its
own.

Fortress regression-checked after the shared xacro changes: gpu_lidar and
rgbd_camera still present, wheel joints still continuous, fdir1 friction intact,
no footprint inertial added, and the robot still drives 0.6 m forward, strafes
cleanly and rotates its wheels.

Co-Authored-By: Claude Opus 5 (1M context) <noreply@anthropic.com>
Claude-Session: https://claude.ai/code/session_01EdVYHU8DgpEjDU7fB4CNqR

* Give the macOS backend its own folder with one entry point

Everything a Mac user needs now lives in yahboom_robostack_M_silycon/: the
launch files, the world, the RViz layout, the environment fixes, a setup
checker, and a guide written for a student rather than a maintainer. A single
./run script drives the whole workflow, so nobody has to know pixi environments,
colcon invocations or which launch file lives in which package.

The Classic launch files, world and RViz config moved here from
yahboom_rosmaster_gazebo rather than being copied, so there is still one source
of truth. They resolve their own assets relative to the folder instead of a
package share, since ros2 launch accepts a path and the folder name cannot be a
ROS package (package names must be lowercase). The root pixi tasks now point at
the new locations and still work.

Also make ./run stop actually stop everything: stop_sim.sh missed gzserver,
gzclient and the whole Nav2 and slam_toolbox stack, which then lingered and
poisoned the next run's ROS graph.

Document that an area must be mapped before Nav2 will navigate into it. A goal
in unmapped space makes the planner return a trivial path and Nav2 reports
success without moving, which looks like a bug and is not.

Verified from a clean build through ./run: drives 0.591 m, strafes the same
sideways, LiDAR returns, and after touring the room Nav2 reaches a goal 2 m away
to within 0.01 m.

Co-Authored-By: Claude Opus 5 (1M context) <noreply@anthropic.com>
Claude-Session: https://claude.ai/code/session_01EdVYHU8DgpEjDU7fB4CNqR

* make simulation better and closer to reality

* Make Tadeo's better-simulation work on the macOS backend

The retuned LiDAR broke Gazebo Classic outright. Dropping range_min from
0.20 to 0.05 m removed an accidental shield: Classic's CPU raycast starts
each ray at range_min, and the chassis collision box spans x [-0.181,
0.119], y +/-0.069, z [0.008, 0.205] about base_link, so the new mount at
(0.043, 0, 0.110) sits inside it. Every one of the 1080 beams returned the
robot's own hull, 0.057-0.242 m, and SLAM and Nav2 were both dead. The old
0.20 m happened to exceed all four faces of the old mount; reverting to it
would not help either, because the new mount puts the rear face at 0.224 m.
Classic now takes 0.25 m, which clears the 0.2345 m rear corner. Fortress
renders from the visual mesh, which the mount clears, so it keeps the
sensor's true 0.05 m.

Verified on an M4 Max: 1080 beams, no returns under 0.25 m, opposite beams
spanning 5.905 m across a 5.90 m room, and a front/rear asymmetry of 0.083 m
against the 0.086 m the 0.043 m offset predicts. slam_toolbox builds a
119x119 map at 0.05 m/cell and Nav2 drives to a goal 1.5 m away and stops
0.10 m from it.

Also on the macOS side, /cmd_vel now runs through cmd_vel_watchdog, so the
Mac gets the same per-direction drift as the Fortress reference instead of
silently skipping it; planar_move reads its output through the new
cmd_vel_topic argument, and motion_bias:=false restores the ideal base.

Three defects in the incoming branch, none of them macOS-specific:

* cmd_vel_watchdog.py and wheel_state_odometry.py were added to
  install(PROGRAMS) as mode 100644. A plain colcon build copies them and
  CMake adds +x to the copy, which hides it; with --symlink-install, which
  this repo uses, the install tree symlinks the source and ros2 launch
  rejects the node as not found. Both are 100755 now.
* lidar_geometry_probe.py still encoded the old contract: 720 samples,
  0.20/30.0 ranges, and a laser frame aligned with base_link. It now models
  the pi yaw and the 0.043 m offset, selects sectors with a wrap-aware
  angular difference because the front target sits on the +/-pi seam, and
  corrects the positive-y residual, whose old form both dropped the offset
  and had the wrong sign.
* The Fortress launch injected randomly sampled drift unconditionally,
  which made motion_profile_divergence_ideal's error <= 0.0005 m assertion
  irreproducible. Gated behind a motion_bias argument, default true, and
  that test now passes motion_bias:=false.

stop_sim.sh missed the topic_tools throttle, which survives as a bare
binary and re-registers joint_state_throttle on the next run, and doctor.sh
now checks the executable bits and motion_bias.yaml.

The Fortress tests were not executed: they need Linux and a renderer.

Co-Authored-By: Tadeo-Casiraghi <tadeo.casiraghi@gmail.com>
Co-Authored-By: Claude Opus 5 <noreply@anthropic.com>
Claude-Session: https://claude.ai/code/session_018MENGNNdhNmtDZsDatQtzn

* add calculated odometry, change file permissions, add gorund truth tf

* updated readme

* Add a from-scratch macOS setup guide for students

The folder README assumes pixi is already installed and the repository is
already cloned, which is exactly the part a student starting from a fresh
Mac does not have. SETUP.md covers that gap end to end: Xcode Command Line
Tools, Homebrew, pixi, which repository to clone, the environment install,
the build, and the first drive, plus how to tell the simulation is actually
healthy and how to remove it again.

Two things it states that people get wrong. The macOS folder only exists on
the fork until pull request #2 lands, so cloning AIRclub-UdeSA gives a tree
without it. And the environment is 4.3 GB installed, not the ~3 GB the
README claimed.

Co-Authored-By: Claude Opus 5 <noreply@anthropic.com>
Claude-Session: https://claude.ai/code/session_018MENGNNdhNmtDZsDatQtzn

* Point Mac users at the macOS folder from the root README

The README rewrite dropped the macOS section and left "Gazebo Classic is not
supported", which is now the opposite of what a Mac user needs to read: the
repository does contain a Classic backend, and on macOS it is the only one
that runs. Scoped that statement to the Linux mecanum simulator and linked
the folder and its setup guide.

Also fixed the clone command, which was missing "clone".

* Stop the ground-truth probe from breaking every Fortress launch test

ground_truth_contract_probe.py had been turned into a runtime TF broadcaster:
complete() was commented out and made to return False "so the node runs
indefinitely", and the Fortress launch started it as a node. That gave one
file two incompatible jobs. As a probe it no longer validated or exited, so
its own contract test failed; and because the shared Fortress launch started
it, every launch test including that file inherited a process that always
exits non-zero, failing test_all_processes_exit_cleanly.

Split the roles. The probe is restored to its validating form, and the TF
broadcast moves to a new scripts/ground_truth_tf.py runtime node publishing
odom -> ground_truth_base from /ground_truth/odom, which is what the launch
now starts. Tadeo's /calc_odom node is untouched.

Also cleared the linters this branch introduced: trailing whitespace, a
missing final newline and an over-long line in calculated_odometry.py, the
stray inline comment in the launch, and two D213 docstrings of mine that put
the summary on the first line where this package puts it on the second.

Measured on Linux with Gazebo Fortress 6.18 under Xvfb/llvmpipe, against
da87ef0 as the baseline:

  lidar_geometry                    FAIL/FAIL -> pass/pass
  imu_motion                        clean-exit regression fixed
  motion_profile_divergence ideal   clean-exit regression fixed
  motion_profile_divergence stress  clean-exit regression fixed
  ground_truth_contract             restored to its baseline result
  flake8                            18 failures -> 0
  pep257                             2 failures -> 0

Totals went 44 failures of 77 to 13 of 61, against 16 of 59 at baseline.
Every remaining failure is identical to baseline, test for test:
base_feedback and depth_geometry clean-exit, depth_geometry probe, and both
sensor_contract worlds. Those predate this branch and are untouched here.

Co-Authored-By: Claude Opus 5 <noreply@anthropic.com>
Claude-Session: https://claude.ai/code/session_018MENGNNdhNmtDZsDatQtzn

* Revert all of Tadeo's changes, back to the pre-better-simulation backend

Restores the tree to b3cda7a, the last commit before better-simulation was
merged. This drops the retuned LiDAR (back to 720 beams at 0.20-30.0 m,
mounted at 0 0 0.0825 with no yaw), the motion-bias drift model and its
config, calculated_odometry.py, the ground-truth TF node, and the README
rewrite. The macOS fixes that only existed to make that work behave on a
Mac go with it, since there is nothing left for them to correct: the
Classic min_range gate, the cmd_vel_topic indirection, the Fortress
motion_bias argument and the lidar_geometry_probe contract repair.

Kept two things that were never Tadeo's: SETUP.md, with its LiDAR
expectations corrected back to 720 beams at 0.20-30.0 m and the drift
section removed, and the stop_sim.sh pattern for the topic_tools throttle,
which is an independent teardown bug.

Local only - not pushed. fork/main still has the full history.

* Reapply Tadeo's simulation work incrementally, with the Mac kept working

Applied his changes one at a time, running the macOS Classic backend after
each, which located two defects precisely.

The LiDAR mount is the first. Moving it to 0.043 0 0.110 puts it inside the
chassis collision box, whose furthest corner is 0.2345 m away. Classic's CPU
raycast starts each ray at range_min rather than clamping, so any range_min
below that begins part of the sweep inside the hull. Applying the mount alone,
with range_min still at the old 0.20, already broke it: 80 of 720 beams came
back under 0.30 m and the room measured 3.14 m across instead of 5.90. His
range_min of 0.05 does not cause this, it takes it from 11% of beams to all of
them. Classic now gates range_min to 0.25 m; Fortress renders from the visual
mesh, which the mount clears, so it keeps his 0.05.

The second is the ground-truth node. ground_truth_contract_probe.py validates
and exits, so launching it as a permanent node left a process that always exits
non-zero and broke test_all_processes_exit_cleanly in every launch test that
includes the Fortress launch file. Split into a ground_truth_tf.py runtime node
with the probe left as a probe.

Everything else of his is in as written: the 1080-beam scan at 12 m with a
tenth the noise, the commented-out LiDAR visual, motion_bias.yaml and the
per-direction drift in the watchdog, calculated_odometry.py and /calc_odom.
The Mac additionally routes /cmd_vel through the watchdog, which his branch
only did for Fortress, so a student on macOS gets the same drift.

Two things his commits would have failed CI on regardless of platform: the new
scripts were added to install(PROGRAMS) at mode 100644, which breaks
--symlink-install because the install tree symlinks the source, and flake8
flagged 19 issues across cmd_vel_watchdog.py and calculated_odometry.py. Both
fixed. The randomised drift also made motion_profile_divergence_ideal's
error <= 0.0005 m assertion irreproducible, so that test now passes
motion_bias:=false against a new launch argument.

Verified on an M4 Max at every step: 1080 beams, no returns under 0.30 m, room
spanning 5.89-5.92 m against a true 5.90, drive and strafe at 0.574 m,
slam_toolbox mapping and Nav2 reaching a goal 1.4 m away to within 0.095 m.
flake8 clean and motion_profile_contract's 4 tests pass. The Fortress launch
tests still need Linux and were not run.

Co-Authored-By: Tadeo-Casiraghi <tadeo.casiraghi@gmail.com>
Co-Authored-By: Claude Opus 5 <noreply@anthropic.com>

* Sync the macOS guide with the reintegrated LiDAR and drift model

The revert had rolled SETUP.md back to 720 beams at 0.20-30.0 m and dropped
the drift section. Reapplying Tadeo's work restored 1080 beams at 0.25-12.0 m
and the motion bias, so a student following the verification table would have
read the live scan and concluded the simulation was broken.

* Fix the two pep257 failures the launch-test run surfaced

Running the suite on macOS found D213 in two docstrings I had written: the
Fortress launch's _rviz_config_for_platform and the LiDAR probe's
x_face_range. The repo's convention starts a multi-line summary on the second
line. flake8, pep257, lint_cmake and xmllint now all pass.

---------

Co-authored-by: Claude Opus 5 (1M context) <noreply@anthropic.com>
Co-authored-by: Tadeo-Casiraghi <tadeo.casiraghi@gmail.com>

File: yahboom_rosmaster_description/urdf/robots/rosmaster_x3.urdf.xacro (robot description, xacro)
@@ -7,4 +7,26 @@
   <xacro:arg name="prefix" default=""/>
   <xacro:arg name="use_gazebo" default="false"/>
+  <!-- Rendering sensors (gpu_lidar, rgbd_camera) need the ogre2 pipeline, which
+       the Gazebo Fortress server cannot initialise on macOS. Set false there to
+       keep the robot, its links and TF while omitting those two sensors. -->
+  <xacro:arg name="render_sensors" default="true"/>
+  <!-- gz_ros2_control only reports joint state here; MecanumDrive owns motion.
+       Activating a controller aborts the Gazebo server on macOS because
+       ros2_control waits on a condition variable holding an unlocked mutex,
+       which libc++ rejects. Set false to publish joint state straight from
+       Gazebo instead and skip ros2_control entirely. -->
+  <xacro:arg name="use_ros2_control" default="true"/>
+  <!-- Which simulator the Gazebo tags target. "fortress" is the upstream
+       backend. "classic" is for macOS, where Fortress cannot render sensors or
+       open its GUI; Gazebo Classic can, and its CPU raycast lidar works there. -->
+  <xacro:arg name="sim_backend" default="fortress"/>
+  <xacro:property name="backend" value="$(arg sim_backend)"/>
+  <!-- Gazebo Classic plugin suffix: conda installs .dylib on macOS, .so on Linux. -->
+  <xacro:arg name="plugin_ext" default=".so"/>
+  <!-- Topic planar_move drives from on the Classic backend. Fortress routes
+       /cmd_vel through cmd_vel_watchdog to add per-direction drift; pointing
+       this at the watchdog's output gives Classic the same treatment, while the
+       default keeps planar_move on /cmd_vel when no watchdog runs. -->
+  <xacro:arg name="cmd_vel_topic" default="cmd_vel"/>
   <!-- Contact parameters are supplied by the simulator motion profile. These
        defaults preserve the ideal description when xacro is expanded directly. -->
@@ -21,5 +43,7 @@
   <xacro:include filename="$(find yahboom_rosmaster_description)/urdf/sensors/lidar.urdf.xacro"/>
   <xacro:include filename="$(find yahboom_rosmaster_description)/urdf/sensors/imu.urdf.xacro"/>
-  <xacro:rosmaster_x3_base prefix="$(arg prefix)"/>
+  <xacro:rosmaster_x3_base
+    prefix="$(arg prefix)"
+    footprint_inertial="${backend == 'classic'}"/>
   <!-- fdir1 = roller grip direction in base_footprint frame via ignition:expressed_in.
        Matches the official Gazebo mecanum demo (expressed_in="chassis", same topology).
@@ -35,5 +59,7 @@
     mu2="$(arg wheel_mu2)"
     slip1="$(arg front_left_slip1)"
-    slip2="$(arg wheel_slip2)"/>
+    slip2="$(arg wheel_slip2)"
+    simple_friction="${backend == 'classic'}"
+    joint_type="${'fixed' if backend == 'classic' else 'continuous'}"/>
   <xacro:mecanum_wheel
     prefix="$(arg prefix)"
@@ -45,5 +71,7 @@
     mu2="$(arg wheel_mu2)"
     slip1="$(arg front_right_slip1)"
-    slip2="$(arg wheel_slip2)"/>
+    slip2="$(arg wheel_slip2)"
+    simple_friction="${backend == 'classic'}"
+    joint_type="${'fixed' if backend == 'classic' else 'continuous'}"/>
   <xacro:mecanum_wheel
     prefix="$(arg prefix)"
@@ -55,5 +83,7 @@
     mu2="$(arg wheel_mu2)"
     slip1="$(arg back_left_slip1)"
-    slip2="$(arg wheel_slip2)"/>
+    slip2="$(arg wheel_slip2)"
+    simple_friction="${backend == 'classic'}"
+    joint_type="${'fixed' if backend == 'classic' else 'continuous'}"/>
   <xacro:mecanum_wheel
     prefix="$(arg prefix)"
@@ -65,20 +95,34 @@
     mu2="$(arg wheel_mu2)"
     slip1="$(arg back_right_slip1)"
-    slip2="$(arg wheel_slip2)"/>
+    slip2="$(arg wheel_slip2)"
+    simple_friction="${backend == 'classic'}"
+    joint_type="${'fixed' if backend == 'classic' else 'continuous'}"/>
   <xacro:rgbd_camera
     prefix="$(arg prefix)"
     camera_name="cam_1"
     xyz_offset="0.105 0 0.05"
-    rpy_offset="0 0 0"/>
+    rpy_offset="0 0 0"
+    enable_gz_sensor="${backend == 'fortress' and '$(arg render_sensors)' in ['true', 'True', '1']}"/>
+  <!-- Classic's CPU raycast starts each ray at range_min, so anything nearer is
+       skipped rather than clamped. The chassis collision box spans x [-0.181,
+       0.119], y +/-0.069, z [0.008, 0.205] about base_link and so encloses this
+       mount, putting its furthest corner 0.2345 m away. Any range_min below
+       that starts part of the sweep inside the hull and those beams return the
+       robot instead of the room. Fortress renders from the visual mesh, which
+       the mount clears, so it keeps the sensor's true minimum. -->
   <xacro:lidar_sensor
     prefix="$(arg prefix)"
     parent="base_link"
     frame_id="laser_frame"
-    xyz_offset="0 0 0.0825"
-    rpy_offset="0 0 0"
+    xyz_offset="0.043 0 0.110"
+    rpy_offset="0 0 ${M_PI}"
+    min_range="${0.25 if backend == 'classic' else 0.05}"
     mesh_xyz_offset="0 0 0"
     mesh_rpy_offset="${-M_PI/2} 0 0"
     update_rate="5"
-    topic_name="scan"/>
+    topic_name="scan"
+    enable_gz_sensor="${backend == 'fortress' and '$(arg render_sensors)' in ['true', 'True', '1']}"
+    classic_sensor="${backend == 'classic'}"
+    plugin_ext="$(arg plugin_ext)"/>
   <xacro:imu_sensor
     prefix="$(arg prefix)"
@@ -91,9 +135,46 @@
   <!-- Gazebo Fortress simulation plugins. gz_ros2_control is read-only for
        wheel and IMU state; native MecanumDrive owns wheel velocity commands. -->
-  <xacro:if value="$(arg use_gazebo)">
+  <xacro:if value="${backend == 'classic'}">
     <gazebo>
-      <plugin filename="gz_ros2_control-system" name="gz_ros2_control::GazeboSimROS2ControlPlugin">
-        <parameters>$(find yahboom_rosmaster_gazebo)/config/ros2_control.yaml</parameters>
+      <!-- ODE parks resting bodies, and a parked body ignores the velocity
+           planar_move sets, so the robot never starts moving. -->
+      <allow_auto_disable>false</allow_auto_disable>
+      <!-- Holonomic base drive. planar_move consumes linear.x, linear.y and
+           angular.z, so it reproduces mecanum strafing, and it owns both /odom
+           and the odom->base_footprint transform. -->
+      <plugin name="planar_move" filename="libgazebo_ros_planar_move$(arg plugin_ext)">
+        <ros>
+          <remapping>cmd_vel:=$(arg cmd_vel_topic)</remapping>
+          <remapping>odom:=odom</remapping>
+        </ros>
+        <update_rate>50</update_rate>
+        <publish_odom>true</publish_odom>
+        <publish_odom_tf>true</publish_odom_tf>
+        <odometry_frame>odom</odometry_frame>
+        <robot_base_frame>$(arg prefix)base_footprint</robot_base_frame>
+        <covariance_x>0.0001</covariance_x>
+        <covariance_y>0.0001</covariance_y>
+        <covariance_yaw>0.01</covariance_yaw>
       </plugin>
+      <!-- No joint state publisher here: the wheels are welded on this backend,
+           so there is nothing to report and robot_state_publisher emits their
+           transforms on /tf_static instead. -->
+    </gazebo>
+  </xacro:if>
+  <xacro:if value="${backend == 'fortress' and '$(arg use_gazebo)' in ['true', 'True', '1']}">
+    <gazebo>
+      <xacro:if value="$(arg use_ros2_control)">
+        <plugin filename="gz_ros2_control-system" name="gz_ros2_control::GazeboSimROS2ControlPlugin">
+          <parameters>$(find yahboom_rosmaster_gazebo)/config/ros2_control.yaml</parameters>
+        </plugin>
+      </xacro:if>
+      <!-- Same wheel-state source as joint_state_broadcaster, published by
+           Gazebo itself. ros_gz_bridge turns it into /joint_states. -->
+      <xacro:unless value="$(arg use_ros2_control)">
+        <plugin filename="ignition-gazebo-joint-state-publisher-system"
+                name="ignition::gazebo::systems::JointStatePublisher">
+          <topic>joint_states_gz</topic>
+        </plugin>
+      </xacro:unless>
       <plugin filename="ignition-gazebo-mecanum-drive-system"
               name="ignition::gazebo::systems::MecanumDrive">
