Commit message: Standardize canonical laser_link frame across URDF, probes, and rviz
- Set frame_id to laser_link in lidar.urdf.xacro and rosmaster_x3.urdf.xacro
- Update sensor_contract_probe and lidar_geometry_probe to assert laser_link
- Update RViz configurations, contract notes, and documentation

File: yahboom_rosmaster_description/urdf/robots/rosmaster_x3.urdf.xacro (robot description, xacro)
@@ -114,5 +114,5 @@
     prefix="$(arg prefix)"
     parent="base_link"
-    frame_id="laser_frame"
+    frame_id="laser_link"
     xyz_offset="0.043 0 0.110"
     rpy_offset="0 0 ${M_PI}"

File: yahboom_rosmaster_description/urdf/sensors/lidar.urdf.xacro (robot description, xacro)
@@ -5,5 +5,5 @@
     prefix:=''
     parent:='base_link'
-    frame_id:='laser_frame'
+    frame_id:='laser_link'
     mesh_file:='file://$(find yahboom_rosmaster_description)/meshes/rplidar/rplidar_s2.stl'
     xyz_offset:='0.043 0 0.110'
@@ -44,15 +44,4 @@
     <xacro:property name="izz" value="${(mass/2) * (radius * radius)}" />
     <link name="${prefix}${frame_id}">
-      <!--
-      <visual>
-        <origin xyz="${mesh_xyz_offset}" rpy="${mesh_rpy_offset}"/>
-        <geometry>
-          <mesh filename="${mesh_file}" scale="${mesh_scale}"/>
-        </geometry>
-        <material name="${material_name}">
-          <color rgba="${material_color}"/>
-        </material>
-      </visual>
-      -->
       <xacro:if value="${enable_collision}">
         <collision>
@@ -79,11 +68,4 @@
       <child link="${prefix}${frame_id}" />
       <origin xyz="${xyz_offset}" rpy="${rpy_offset}"/>
-    </joint>
-    <!-- Alias link: provides laser_link in TF for stacks expecting laser_link rather than laser_frame -->
-    <link name="${prefix}laser_link"/>
-    <joint name="${prefix}laser_link_alias_joint" type="fixed">
-      <parent link="${prefix}${frame_id}"/>
-      <child link="${prefix}laser_link"/>
-      <origin xyz="0 0 0" rpy="0 0 0"/>
     </joint>
     <gazebo reference="${prefix}${frame_id}">

Commit message: feat: model the physical X3's Astra camera
The simulated RGB-D camera ran at 424x240, 5 Hz and 87 deg, rendered
from cam_1_link, and labelled its four image and camera_info topics
cam_1_depth_optical_frame. The physical X3's Astra publishes both
streams at 320x240 and 30 Hz. They use its color intrinsics:
fx = fy = 271.809, cx = 158.719, cy = 120.092, plumb_bob with zero D
(physical_rosmaster camera_public.json). Depth is registered to color,
so every topic carries cam_1_color_optical_frame.

Breaking for teams: resolution, field of view (60.97 deg), rate and
frame labels all change.

rgbd_camera.urdf.xacro now takes the calibrated focal length and
derives the horizontal FOV Gazebo renders from, 1.0640610 rad. The
sensor moves to cam_1_color_frame. URDF-to-SDF lumping carries its
25.1 mm offset and 0.34 deg rotation into the sensor pose.

The principal point is not configurable. Fortress writes <intrinsics>
and <projection> into camera_info, but Ogre2DepthCamera never applies
them and renders a symmetric frustum. (158.719, 120.092), (160, 120)
and (140, 100) produced bit-identical images. Gazebo's own cloud rays
put the frustum's axis at (159.5, 119.5) in ROS pixel coordinates, and
the target's edges in the depth image land on the pixels that predicts.
Publish that point, 0.78 and 0.59 px from physical. Gazebo's default
of width / 2 is half a pixel off its own image.

Gazebo's cloud is expressed in the sensor's regular frame, now
cam_1_color_frame. Relabelling it cam_1_depth_frame, as
pointcloud_frame_relay.py did, would leave it 25 mm off, so the relay
transforms every finite point with the static cam_1_depth_frame <-
cam_1_color_frame transform from /tf_static, as the physical
sensor_adapter.py does. Its arithmetic stays element-wise: a numpy
matrix product ran on a multithreaded BLAS whose spinning threads took
8.5 cores and cut the real-time factor to 0.77. On the host GPU the
transform costs 1.6 ms per cloud, which moves the cloud from 27.1 to
25.2 Hz against the relabel-only relay.

The ledger's step-5 entries now match physical: the four frame_id and
rate_hz entries (contract 27-33 Hz; the stamps run at 30.3 Hz with the
1 ms physics step), camera.width, fx, fy, cx, cy (tolerances 0.8 and
0.6 px) and horizontal_fov_rad. The cloud's rate contract moves to
27-33 Hz and stays a step-6 gap.

sensor_contract_probe checks camera_info against the ledger's
intrinsics, image size and distortion instead of a centred principal
point. depth_geometry measures the target from the color aperture
(0.745 m). It requires the red target's centroid where that aperture
sees it (169.5 px, against 159.5 px from the depth aperture). It also
requires each sampled cloud point within 5 mm of the depth image's
point transformed into cam_1_depth_frame. The relabel-only relay fails
that check by 25 mm, and a camera left at cam_1_link fails the parallax
check. The description contract finds the sensor on cam_1_color_frame
and checks its frame labels and projection.

Refs #43

File: yahboom_rosmaster_description/urdf/robots/rosmaster_x3.urdf.xacro (robot description, xacro)
@@ -104,5 +104,7 @@
        factory calibration of one unit, Astra serial ACRC64300ET: the color
        sensor sits 25.1 mm left of depth, and another unit differs slightly.
-       yahboom_rosmaster_gazebo/config/real_robot_contract.yaml records both. -->
+       Gazebo renders both images from the color frame, as the Astra registers
+       depth to color. yahboom_rosmaster_gazebo/config/real_robot_contract.yaml
+       records both frames. -->
   <xacro:rgbd_camera
     prefix="$(arg prefix)"

File: yahboom_rosmaster_description/urdf/sensors/rgbd_camera.urdf.xacro (robot description, xacro)
@@ -31,22 +31,31 @@
     iyz:=0.0
     izz:=0.003879257
-    horizontal_fov:=1.5184
-    image_width:=424
+    focal_length:=271.80938720703125
+    image_width:=320
     image_height:=240
     clip_near:=0.05
     clip_far:=8.0
-    update_rate:=5
+    update_rate:=30
     always_on:=1
     visualize:=false
     enable_collision:=false
     enable_gz_sensor:=true">
-    <!-- Fortress 6.8 populates RGB-D CameraInfo before configuring the
-         renderer, so its implicit values remain the SDFormat 320x240 defaults
-         (fx=fy=277, cx=160, cy=120). Publish intrinsics that actually match
-         this image size and horizontal FOV. -->
-    <xacro:property name="focal_length"
-                    value="${image_width / (2.0 * tan(horizontal_fov / 2.0))}" />
-    <xacro:property name="principal_x" value="${image_width / 2.0}" />
-    <xacro:property name="principal_y" value="${image_height / 2.0}" />
+    <!-- The defaults are the physical X3's Astra: both streams at 320x240 and
+         30 Hz with the color intrinsics, to which the driver registers depth
+         (physical_rosmaster robot_artifacts/x3c_sensor_capability_2026-09-17/
+         camera_public.json). Gazebo renders from the horizontal FOV, so it is
+         derived from the focal length.
+         The principal point is not a parameter. Fortress copies <intrinsics>
+         and <projection> into CameraInfo, but its RGB-D camera
+         (Ogre2DepthCamera) never applies them and always renders a symmetric
+         frustum: an off-centre or deliberately wrong principal point changes
+         CameraInfo and leaves the image bit-identical. With ROS pixel centres
+         at integer coordinates, that frustum's axis is at ((width - 1) / 2,
+         (height - 1) / 2). Publish that, not Gazebo's own width / 2, which is
+         half a pixel off the rendered image. -->
+    <xacro:property name="horizontal_fov"
+                    value="${2.0 * atan(image_width / (2.0 * focal_length))}" />
+    <xacro:property name="principal_x" value="${(image_width - 1) / 2.0}" />
+    <xacro:property name="principal_y" value="${(image_height - 1) / 2.0}" />
     <link name="${prefix}${camera_name}_link">
       <visual>
@@ -90,6 +99,6 @@
     <!-- The color frames sit at the color sensor's offset from cam_1_link, as
          the physical Astra driver publishes them. The Fortress rgbd_camera
-         still renders color and depth from one aperture at cam_1_link and
-         labels both with the depth optical frame. -->
+         below renders color and depth from this one aperture: the Astra
+         registers depth to color, so its depth image is also seen from here. -->
     <joint name="${prefix}${camera_name}_color_joint" type="fixed">
       <origin xyz="${color_xyz_offset}" rpy="${color_rpy_offset}" />
@@ -108,5 +117,5 @@
          by the world. Data is bridged to ROS by ros_gz_bridge and ros_gz_image.
          libgazebo_ros_camera.so is Classic-only and must NOT be used here. -->
-    <gazebo reference="${prefix}${camera_name}_link">
+    <gazebo reference="${prefix}${camera_name}_color_frame">
       <!-- See lidar.urdf.xacro: the ogre2 render pipeline cannot initialise in
            the Gazebo server's render thread on macOS. -->
@@ -118,5 +127,5 @@
                the native XYZ point cloud and label image/calibration data
                with the optical frame through SDFormat's dedicated field. -->
-          <optical_frame_id>${prefix}${camera_name}_depth_optical_frame</optical_frame_id>
+          <optical_frame_id>${prefix}${camera_name}_color_optical_frame</optical_frame_id>
           <horizontal_fov>${horizontal_fov}</horizontal_fov>
           <image>
@@ -153,5 +162,5 @@
         <visualize>${visualize}</visualize>
         <topic>${prefix}${camera_name}</topic>
-        <gz_frame_id>${prefix}${camera_name}_depth_frame</gz_frame_id>
+        <gz_frame_id>${prefix}${camera_name}_color_frame</gz_frame_id>
       </sensor>
       </xacro:if>

Commit message: feat(gazebo): publish /imu/data_raw as the robot's driver does and estimate /imu/data with imu_filter_madgwick (#43 step 8c)
- The IMU's per-axis noise is the physical robot's stationary capture under the
  physical sensor profile and zero under ideal. The launch passes the selected
  profile's values to the description as xacro arguments; the xacro defaults are
  the physical values, and a test keeps them equal to sensor_profiles.yaml.
- imu_raw_relay.py republishes the bridged IMU as /imu/data_raw with exactly the
  content of the driver's message: the identity quaternion, zero covariances,
  Reliable, depth 100.
- The stock imu_filter_madgwick node, with the five parameters of the robot's
  imu_filter_param.yaml, produces /imu/data under both profiles. The package
  depends on it.
- imu_motion_probe reads its expectations from the ledger, expresses the
  orientation in base_link through TF, judges yaw as a change, and grades the
  raw stream's content and the per-axis noise. New launch targets imu_noise and
  imu_motion_physical; imu_motion runs under ideal.

File: yahboom_rosmaster_description/urdf/robots/rosmaster_x3.urdf.xacro (robot description, xacro)
@@ -38,4 +38,15 @@
   <xacro:arg name="back_left_slip1" default="0.0"/>
   <xacro:arg name="back_right_slip1" default="0.0"/>
+  <!-- Per-axis IMU noise, in imu_link. The defaults are the physical robot's
+       stationary capture, so a standalone render (and the description synced to
+       other repositories) is the `physical` sensor profile. The simulator launch
+       passes the selected profile's values from config/sensor_profiles.yaml,
+       zeros for `ideal`; a test keeps these defaults equal to that file. -->
+  <xacro:arg name="imu_gyro_noise_stddev_x" default="0.0054"/>
+  <xacro:arg name="imu_gyro_noise_stddev_y" default="0.0051"/>
+  <xacro:arg name="imu_gyro_noise_stddev_z" default="0.0052"/>
+  <xacro:arg name="imu_accel_noise_stddev_x" default="0.135"/>
+  <xacro:arg name="imu_accel_noise_stddev_y" default="0.131"/>
+  <xacro:arg name="imu_accel_noise_stddev_z" default="0.102"/>
   <xacro:include filename="$(find yahboom_rosmaster_description)/urdf/mech/rosmaster_x3_base.urdf.xacro"/>
   <xacro:include filename="$(find yahboom_rosmaster_description)/urdf/mech/mecanum_wheel.urdf.xacro"/>
@@ -143,4 +154,10 @@
     rpy_offset="0 3.1415 1.5707"
     update_rate="10.0"
+    gyro_noise_stddev_x="$(arg imu_gyro_noise_stddev_x)"
+    gyro_noise_stddev_y="$(arg imu_gyro_noise_stddev_y)"
+    gyro_noise_stddev_z="$(arg imu_gyro_noise_stddev_z)"
+    accel_noise_stddev_x="$(arg imu_accel_noise_stddev_x)"
+    accel_noise_stddev_y="$(arg imu_accel_noise_stddev_y)"
+    accel_noise_stddev_z="$(arg imu_accel_noise_stddev_z)"
     topic_name="imu/data"/>
   <!-- Gazebo Fortress simulation plugins. gz_ros2_control is read-only for

File: yahboom_rosmaster_description/urdf/sensors/imu.urdf.xacro (robot description, xacro)
@@ -2,4 +2,11 @@
 <robot xmlns:xacro="http://www.ros.org/wiki/xacro">
     <xacro:property name="M_PI" value="3.1415926535897931" />
+    <xacro:macro name="imu_noise" params="axis stddev">
+        <xacro:if value="${float(stddev) > 0.0}">
+            <xacro:element xacro:name="${axis}">
+                <noise type="gaussian"><mean>0</mean><stddev>${stddev}</stddev></noise>
+            </xacro:element>
+        </xacro:if>
+    </xacro:macro>
     <xacro:macro name="imu_sensor" params="
         prefix:=''
@@ -20,6 +27,10 @@
         gazebo_material_specular:='0.1 0.1 0.1 1'
         update_rate:='10.0'
-        gyro_noise_stddev:='0.00873'
-        accel_noise_stddev:='0.00175'
+        gyro_noise_stddev_x:='0.0054'
+        gyro_noise_stddev_y:='0.0051'
+        gyro_noise_stddev_z:='0.0052'
+        accel_noise_stddev_x:='0.135'
+        accel_noise_stddev_y:='0.131'
+        accel_noise_stddev_z:='0.102'
         topic_name:='imu/data'
         always_on:=true
@@ -68,13 +79,16 @@
             <sensor name="${prefix}imu_sensor" type="imu">
                 <imu>
+                    <!-- Per-axis Gaussian noise, as the physical robot's stationary
+                         capture measured it. A zero standard deviation (sensor_profile
+                         ideal) drops the noise element instead of writing one. -->
                     <angular_velocity>
-                        <x><noise type="gaussian"><mean>0</mean><stddev>${gyro_noise_stddev}</stddev></noise></x>
-                        <y><noise type="gaussian"><mean>0</mean><stddev>${gyro_noise_stddev}</stddev></noise></y>
-                        <z><noise type="gaussian"><mean>0</mean><stddev>${gyro_noise_stddev}</stddev></noise></z>
+                        <xacro:imu_noise axis="x" stddev="${gyro_noise_stddev_x}"/>
+                        <xacro:imu_noise axis="y" stddev="${gyro_noise_stddev_y}"/>
+                        <xacro:imu_noise axis="z" stddev="${gyro_noise_stddev_z}"/>
                     </angular_velocity>
                     <linear_acceleration>
-                        <x><noise type="gaussian"><mean>0</mean><stddev>${accel_noise_stddev}</stddev></noise></x>
-                        <y><noise type="gaussian"><mean>0</mean><stddev>${accel_noise_stddev}</stddev></noise></y>
-                        <z><noise type="gaussian"><mean>0</mean><stddev>${accel_noise_stddev}</stddev></noise></z>
+                        <xacro:imu_noise axis="x" stddev="${accel_noise_stddev_x}"/>
+                        <xacro:imu_noise axis="y" stddev="${accel_noise_stddev_y}"/>
+                        <xacro:imu_noise axis="z" stddev="${accel_noise_stddev_z}"/>
                     </linear_acceleration>
                 </imu>
