Commit message: Add laser_link TF alias and graceful zero-stop in cmd_vel_watchdog
- Add laser_link alias link and joint in lidar.urdf.xacro for physical_rosmaster parity
- Add fail-safe zero-velocity stop on shutdown in cmd_vel_watchdog.py

File: yahboom_rosmaster_description/urdf/sensors/lidar.urdf.xacro (robot description, xacro)
@@ -79,4 +79,11 @@
       <child link="${prefix}${frame_id}" />
       <origin xyz="${xyz_offset}" rpy="${rpy_offset}"/>
+    </joint>
+    <!-- Alias link: provides laser_link in TF for stacks expecting laser_link rather than laser_frame -->
+    <link name="${prefix}laser_link"/>
+    <joint name="${prefix}laser_link_alias_joint" type="fixed">
+      <parent link="${prefix}${frame_id}"/>
+      <child link="${prefix}laser_link"/>
+      <origin xyz="0 0 0" rpy="0 0 0"/>
     </joint>
     <gazebo reference="${prefix}${frame_id}">

Commit message: Refactor into dedicated simulator bringup workspace with real-robot parity (#4)
* Add real-robot bag analyzer and interface contract

Protects bags_x3.zip from Git, adds a reusable rosbag2_py analyzer that
derives topic/frame/rate/geometry/noise statistics directly from recorded
bags without full playback, and commits the resulting real_robot_contract.yaml
with per-section confidence and explicit calibration gaps (no ground truth,
no usable encoder feedback in these recordings).

* Fix wheel-separation mismatch and add real-robot IMU mount parity

Reconciles an internal inconsistency: the visual/collision URDF already
used the correct 0.169m wheel separation, but the MecanumDrive plugin and
wheel_state_odometry.py both drove kinematics off a stale 0.149m. The
plugin now references the shared xacro property instead of duplicating it.

Also mounts the IMU at the real robot's measured extrinsic and rate
(10Hz, offset/rotated per real_robot_contract.yaml), which flips which
sensor axis reports gravity, body accel, and yaw rate -- imu_motion_probe.py
is updated to check the correctly mapped sensor axes instead of assuming
an identity mount.

LiDAR parity (1080 rays, 0.05-12m range, laser_link frame, real mount
offset) was attempted and reverted: it reproducibly makes Gazebo Fortress's
gpu_lidar sensor blind (zero finite returns anywhere in the scan, including
targets placed directly in its path), confirmed independently from both the
nonzero X/Y mount offset and the ray-count/range settings alone. Documented
in real_robot_contract.yaml as follow-up work rather than merged broken.

All affected launch tests (lidar_geometry, imu_motion,
motion_profile_divergence_ideal/stress, wheel_odometry_resilience,
sensor_contract_empty/cafe) pass.

* Make dynamic TF contract wait for odometry edge

* Fix real-robot bag analyzer lint

* Refactor repository into dedicated simulator bringup workspace

- Remove navigation, docking, localization, and system_tests demo packages
- Add canonical rosmaster_x3_sim.launch.py bringup entrypoint
- Add Docker environment setup (Dockerfile, container.sh)
- Update metapackage and bringup package declarations
- Streamline macOS pixi tasks and scripts

* Restore environment maps into yahboom_rosmaster_gazebo/maps

- Move cafe_world_map and house_world_map into yahboom_rosmaster_gazebo/maps
- Add maps directory to yahboom_rosmaster_gazebo CMakeLists.txt install rules

* Add laser_link TF alias and graceful zero-stop in cmd_vel_watchdog

- Add laser_link alias link and joint in lidar.urdf.xacro for physical_rosmaster parity
- Add fail-safe zero-velocity stop on shutdown in cmd_vel_watchdog.py

* Standardize canonical laser_link frame across URDF, probes, and rviz

- Set frame_id to laser_link in lidar.urdf.xacro and rosmaster_x3.urdf.xacro
- Update sensor_contract_probe and lidar_geometry_probe to assert laser_link
- Update RViz configurations, contract notes, and documentation

* Fix Gazebo world path resolution and gui/headless launch argument handling

- Add dynamic world path resolver to load local worlds by name (empty.world, cafe.world)
- Add worlds directory to IGN_GAZEBO_RESOURCE_PATH and GZ_SIM_RESOURCE_PATH
- Harmonize gui and headless launch arguments across bringup and gazebo launches

* Relabel Fortress RGB-D point cloud to its true frame

Fortress 6.18 stamps the rgbd_camera PointCloudPacked with the sensor's
optical_frame_id even though its XYZ data stays in the regular +X-forward
camera frame. With the REP-104 optical TF intact, RViz therefore rendered
the cloud rotated about 90 degrees onto the ground plane beside the robot
(a known red box at world (0.9, 0, 0.115) landed at (0.18, -0.695, 0.082)).

Bridge the gz points topic to a private raw topic and relabel its header
to cam_1_depth_frame in pointcloud_frame_relay.py instead of collapsing
the optical rotation: images and CameraInfo keep the optical frame while
the cloud carries the label its coordinates actually use, which restores
absolute alignment and image/cloud registration at the same time.

* Extend RGB-D camera clip range to 8 metres

clip_far 1.5 m cut all rendering well inside the D435 range the sensor
models (rated to ~10 m), so walls vanished from both the color image and
the depth cloud in the cafe world. Pin the depth_geometry probe's far
bound to the same value.

* Move the RGB-D bridge handoff to /internal and document it

Name the private bridge-to-relay topic /internal/cam_1/points_raw so it
reads as an implementation detail instead of looking like a usable
camera topic in RViz, and document the handoff plus why the relay exists
in the README.

* Fix lint regressions in watchdog and relay scripts

File: yahboom_rosmaster_description/urdf/sensors/lidar.urdf.xacro (robot description, xacro)
@@ -5,5 +5,5 @@
     prefix:=''
     parent:='base_link'
-    frame_id:='laser_frame'
+    frame_id:='laser_link'
     mesh_file:='file://$(find yahboom_rosmaster_description)/meshes/rplidar/rplidar_s2.stl'
     xyz_offset:='0.043 0 0.110'
@@ -44,15 +44,4 @@
     <xacro:property name="izz" value="${(mass/2) * (radius * radius)}" />
     <link name="${prefix}${frame_id}">
-      <!--
-      <visual>
-        <origin xyz="${mesh_xyz_offset}" rpy="${mesh_rpy_offset}"/>
-        <geometry>
-          <mesh filename="${mesh_file}" scale="${mesh_scale}"/>
-        </geometry>
-        <material name="${material_name}">
-          <color rgba="${material_color}"/>
-        </material>
-      </visual>
-      -->
       <xacro:if value="${enable_collision}">
         <collision>
