Commit message: Fix RGB-D camera calibration intrinsics

File: yahboom_rosmaster_description/urdf/sensors/rgbd_camera.urdf.xacro (robot description, xacro)
@@ -46,4 +46,12 @@
     visualize:=false
     enable_collision:=false">
+    <!-- Fortress 6.8 populates RGB-D CameraInfo before configuring the
+         renderer, so its implicit values remain the SDFormat 320x240 defaults
+         (fx=fy=277, cx=160, cy=120). Publish intrinsics that actually match
+         this image size and horizontal FOV. -->
+    <xacro:property name="focal_length"
+                    value="${image_width / (2.0 * tan(horizontal_fov / 2.0))}" />
+    <xacro:property name="principal_x" value="${image_width / 2.0}" />
+    <xacro:property name="principal_y" value="${image_height / 2.0}" />
     <link name="${prefix}${camera_name}_link">
       <visual>
@@ -141,4 +149,23 @@
             <far>${clip_far}</far>
           </clip>
+          <lens>
+            <type>gnomonical</type>
+            <scale_to_hfov>true</scale_to_hfov>
+            <intrinsics>
+              <fx>${focal_length}</fx>
+              <fy>${focal_length}</fy>
+              <cx>${principal_x}</cx>
+              <cy>${principal_y}</cy>
+              <s>0.0</s>
+            </intrinsics>
+            <projection>
+              <p_fx>${focal_length}</p_fx>
+              <p_fy>${focal_length}</p_fy>
+              <p_cx>${principal_x}</p_cx>
+              <p_cy>${principal_y}</p_cy>
+              <tx>0.0</tx>
+              <ty>0.0</ty>
+            </projection>
+          </lens>
         </camera>
         <always_on>${always_on}</always_on>

Commit message: feat(description): remove the infra camera frames
The rgbd_camera macro published cam_1_infra1_frame, cam_1_infra2_frame
and their optical frames, inherited from the D435 description it was
written for. The physical X3's Astra driver publishes neither, so a
consumer that looks them up works in the simulator and fails on the
robot. Remove their joints, links and macro parameters, and drop them
from both RViz configs.

This is a TF-visible change: the four frames no longer exist.

Flip the ledger's frames.camera_frames entry to matches_physical, and
remove the frames from the description contract.

Refs #43

File: yahboom_rosmaster_description/urdf/sensors/rgbd_camera.urdf.xacro (robot description, xacro)
@@ -19,8 +19,4 @@
     depth_frame_xyz_offset:='0 0 0'
     depth_frame_rpy_offset:='0 0 0'
-    infra1_xyz_offset:='0 0 0'
-    infra1_rpy_offset:='0 0 0'
-    infra2_xyz_offset:='0 -0.05 0'
-    infra2_rpy_offset:='0 0 0'
     color_xyz_offset:='0 0 0'
     color_rpy_offset:='0 0 0'
@@ -92,28 +88,4 @@
     </joint>
     <link name="${prefix}${camera_name}_depth_optical_frame"/>
-    <joint name="${prefix}${camera_name}_infra1_joint" type="fixed">
-      <origin xyz="${infra1_xyz_offset}" rpy="${infra1_rpy_offset}" />
-      <parent link="${prefix}${camera_name}_link" />
-      <child link="${prefix}${camera_name}_infra1_frame" />
-    </joint>
-    <link name="${prefix}${camera_name}_infra1_frame"/>
-    <joint name="${prefix}${camera_name}_infra1_optical_joint" type="fixed">
-      <origin xyz="${optical_xyz_offset}" rpy="${optical_rpy_offset}" />
-      <parent link="${prefix}${camera_name}_infra1_frame" />
-      <child link="${prefix}${camera_name}_infra1_optical_frame" />
-    </joint>
-    <link name="${prefix}${camera_name}_infra1_optical_frame"/>
-    <joint name="${prefix}${camera_name}_infra2_joint" type="fixed">
-      <origin xyz="${infra2_xyz_offset}" rpy="${infra2_rpy_offset}" />
-      <parent link="${prefix}${camera_name}_link" />
-      <child link="${prefix}${camera_name}_infra2_frame" />
-    </joint>
-    <link name="${prefix}${camera_name}_infra2_frame"/>
-    <joint name="${prefix}${camera_name}_infra2_optical_joint" type="fixed">
-      <origin xyz="${optical_xyz_offset}" rpy="${optical_rpy_offset}" />
-      <parent link="${prefix}${camera_name}_infra2_frame" />
-      <child link="${prefix}${camera_name}_infra2_optical_frame" />
-    </joint>
-    <link name="${prefix}${camera_name}_infra2_optical_frame"/>
     <!-- The Fortress rgbd_camera renders color and depth from one aperture and
          exposes only one optical frame ID.  Keep the color-named frames as
